File: Esquemáticos/ESP32/Motores.kicad_sch (KiCad schematic)
At the start: 11 parts, among them J1 Conector para bobinas del mot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, J2 Conector para bobinas del mot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, U1 ULN2003A, U2 ULN2003A

Commit message: .
Other:
- note added: "NOTA: Este es un concepto inspirado en el módulo para arduino con TLP281"
Changed lines of the file:
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@@
+    (effects (font (size 1.27 1.27)) (justify left bottom))
+  )
+  (text "NOTA: Este es un concepto inspirado en el módulo para arduino con TLP281"
+    (at 53.34 133.35 0)
     (effects (font (size 1.27 1.27)) (justify left bottom))
   )

Commit message: Cambios hechos al esquemático, faltan detalles
Revisar el discord para dejar todo al día con el feedback de hoy
Parts:
- added Q? (x3): S8050, Package_TO_SOT_THT:TO-92_Inline, symbol Transistor_BJT:S8050
- added R? (x6): 5.1k, symbol Device:R
- added R? (x3): 220, symbol Device:R
- added unit 2 of U1
- added unit 3 of U1
- added unit 4 of U1
- gave numbers to parts that had none: 1
Connections:
- net 12V: now also R?.1, R?.1, R?.1, R?.1, R?.1, R?.1
- net GND: now also U1.4, U1.6, U1.8
- net Out2: now also Q?.3 (C), R?.2
- net Out3: now also Q?.3 (C), R?.2
- net Out4: now also Q?.3 (C), R?.2
- new net: Q?.1 (E), U1.13
- new net: Q?.2 (B), R?.2, U1.14
- new net: R?.2, U1.3
- new net: Q?.1 (E), U1.11
- new net: Q?.2 (B), R?.2, U1.12
- new net: R?.2, U1.5
- new net: Q?.2 (B), R?.2, U1.10
- new net: R?.2, U1.7
- new net: Q?.1 (E), U1.9
- new net In2: R?.1
- new net In3: R?.1
- new net In4: R?.1
Other:
- moved on the sheet: Q?, R?, U1A

Commit message: Actualizada la etapa de motores
Parts:
- removed Q? (x4): S8050, Package_TO_SOT_THT:TO-92_Inline, symbol Transistor_BJT:S8050
- removed R? (x8): 5.1k, symbol Device:R
- removed R? (x4): 220, symbol Device:R
- added Q1, Q2, Q3, Q4, Q? (x4): S8050, Package_TO_SOT_THT:TO-92_Inline, symbol Transistor_BJT:S8050
- added R1, R2, R3, R4, R5, R6, R7, R8, R? (x8): 5.1k, symbol Device:R
- added R10, R11, R12, R9, R? (x4): 220, symbol Device:R
- added U? (x4): LTV-247, Package_SO:SOP-16_4.4x10.4mm_P1.27mm, symbol Isolator:LTV-247
Connections:
- net 12V: now also R1.1, R2.1, R3.1, R4.1, R5.1, R6.1, R7.1, R8.1, R?.1, R?.1, R?.1, R?.1, R?.1, R?.1, R?.1, R?.1
- net GND: now also U1.11, U1.13, U1.15, U1.9, Q1.1 (E), Q2.1 (E), Q3.1 (E), Q4.1 (E), Q?.1 (E), Q?.1 (E), Q?.1 (E), Q?.1 (E), U?.11, U?.13, U?.15, U?.9; no longer U1.2, U1.4, U1.6, U1.8
- net In1: now also R9.1
- net In2: now also R10.1
- net In3: now also R11.1
- net In4: now also R12.1
- net Out1: now also Q1.3 (C), R1.2
- net Out2: now also Q2.3 (C), R3.2
- net Out3: now also Q3.3 (C), R5.2
- net Out4: now also Q4.3 (C), R7.2
- net Out5: now also Q?.3 (C), R?.2
- net Out6: now also Q?.3 (C), R?.2
- net Out7: now also Q?.3 (C), R?.2
- net Out8: now also Q?.3 (C), R?.2
- net at U1.14: now also Q2.2 (B), R4.2
- net at U1.3: now also R10.2
- net at U1.12: now also Q3.2 (B), R6.2
- net at U1.5: now also R11.2
- net at U1.10: now also Q4.2 (B), R8.2
- net at U1.7: now also R12.2
- net at U1.1: now also R9.2
- net at U1.16: now also Q1.2 (B), R2.2
- new net: Q?.2 (B), R?.2, U?.10
- new net: Q?.2 (B), R?.2, U?.16
- new net: Q?.2 (B), R?.2, U?.14
- new net: R?.2, U?.3
- new net: Q?.2 (B), R?.2, U?.12
- new net: R?.2, U?.5
- new net: R?.2, U?.7
- new net: R?.2, U?.1
- new net GNDL: U1.2, U1.4, U1.6, U1.8, U?.2, U?.4, U?.6, U?.8
- new net In5: R?.1
- new net In6: R?.1
- new net In7: R?.1
- new net In8: R?.1
Other:
- note added: "NOTA: Este es un diseño inspirado en el módulo para arduino con TLP281"
- note added: "NOTA: Este es un diseño inspirado en el módulo para arduino con ULN2003"
- note added: "Optoacopladores para proteger el resto del sistema"
- note added: "Revisar bien si esto es correcto (Conectar a la tierra común acá)"
- note added: "Revisar bien si esto es correcto (Meter 12V alegremente)"
- note removed: "4 optoacopladores pero solo permite hacer conexiones con 1 de los 4 :/"
- note removed: "NOTA: Este es un concepto inspirado en el módulo para arduino con TLP281"
- note removed: "No entiendo bien por que se supone que este componente contiene"
- note removed: "Optoacopladores para proteger el resto del sistema (provisional)"
- moved on the sheet: C1, C2, J1, J2, U1, U2
