File: Esquemáticos/ESP32/Motores.kicad_sch (KiCad schematic)
At the start: 40 parts, among them J1 Conector para bobinas del mot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, J2 Conector para bobinas del mot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, Q1 S8050, Q2 S8050, Q3 S8050, Q4 S8050, Q5 S8050, Q6 S8050, Q7 S8050, Q8 S8050, U1 LTV-247, U1 ULN2003A, U2 LTV-247, U2 ULN2003A

Commit message: Arreglando los bugs xd
Parts:
- removed C1, C2: 100n, symbol Device:C
- removed J1: Conector para bobinas del motor 1, symbol Connector_Generic:Conn_01x04
- removed J2: Conector para bobinas del motor 2, symbol Connector_Generic:Conn_01x04
- removed Q1, Q2, Q3, Q4, Q5, Q6, Q7, Q8: S8050, Package_TO_SOT_THT:TO-92_Inline, symbol Transistor_BJT:S8050
- removed R1, R13, R14, R15, R16, R17, R18, R19, R2, R20, R3, R4, R5, R6, R7, R8: 5.1k, symbol Device:R
- removed R10, R11, R12, R21, R22, R23, R24, R9: 220, symbol Device:R
- removed U1, U2: LTV-247, Package_SO:SOP-16_4.4x10.4mm_P1.27mm, symbol Isolator:LTV-247
- added C? (x2): 100n, symbol Device:C
- added J?: Conector para bobinas del motor 1, symbol Connector_Generic:Conn_01x04
- added J?: Conector para bobinas del motor 2, symbol Connector_Generic:Conn_01x04
- added Q? (x8): S8050, Package_TO_SOT_THT:TO-92_Inline, symbol Transistor_BJT:S8050
- added R? (x16): 5.1k, symbol Device:R
- added R? (x8): 220, symbol Device:R
- added U? (x2): ULN2003A, symbol Transistor_Array:ULN2003A
- added U? (x8): LTV-247, Package_SO:SOP-16_4.4x10.4mm_P1.27mm, symbol Isolator:LTV-247
Connections:
- net 12V: now also C?.1, C?.1, U?.9 (COM), U?.9 (COM)
- net 5V: now also R?.1, R?.1, R?.1, R?.1, R?.1, R?.1, R?.1, R?.1, R?.1, R?.1, R?.1, R?.1, R?.1, R?.1, R?.1, R?.1
- net GND: now also C?.2, C?.2, Q?.1 (E), Q?.1 (E), Q?.1 (E), Q?.1 (E), Q?.1 (E), Q?.1 (E), Q?.1 (E), Q?.1 (E), U?.11, U?.11, U?.13, U?.13, U?.15, U?.15, U?.8 (GND), U?.8 (GND), U?.9, U?.9
- net GNDL: now also U?.2, U?.2, U?.4, U?.4, U?.6, U?.6, U?.8, U?.8
- net In1: now also R?.1
- net In2: now also R?.1
- net In3: now also R?.1
- net In4: now also R?.1
- net In5: now also R?.1
- net In6: now also R?.1
- net In7: now also R?.1
- net In8: now also R?.1
- net Out1: now also Q?.3 (C), R?.2, U?.1 (I1)
- net Out2: now also Q?.3 (C), R?.2, U?.2 (I2)
- net Out3: now also Q?.3 (C), R?.2, U?.3 (I3)
- net Out4: now also Q?.3 (C), R?.2, U?.4 (I4)
- net Out5: now also Q?.3 (C), R?.2, U?.1 (I1)
- net Out6: now also Q?.3 (C), R?.2, U?.2 (I2)
- net Out7: now also Q?.3 (C), R?.2, U?.3 (I3)
- net Out8: now also Q?.3 (C), R?.2, U?.4 (I4)
- new net: J?.4 (Pin_4), U?.13 (O4) (x2)
- new net: J?.3 (Pin_3), U?.14 (O3) (x2)
- new net: J?.2 (Pin_2), U?.15 (O2) (x2)
- new net: J?.1 (Pin_1), U?.16 (O1) (x2)
- new net: R?.2, U?.7 (x2)
- new net: Q?.2 (B), R?.2, U?.16 (x2)
- new net: R?.2, U?.1 (x2)
- new net: Q?.2 (B), R?.2, U?.14 (x2)
- new net: R?.2, U?.3 (x2)
- new net: Q?.2 (B), R?.2, U?.12 (x2)
- new net: R?.2, U?.5 (x2)
- new net: Q?.2 (B), R?.2, U?.10 (x2)

Commit message: Mas commits :sunglasses:
Agragados números de los componentes
Parts:
- removed Q? (x8): S8050, Package_TO_SOT_THT:TO-92_Inline, symbol Transistor_BJT:S8050
- removed R? (x12): 5.1k, symbol Device:R
- added Q1, Q2, Q3, Q4, Q5, Q6, Q7, Q8: S8550, Package_TO_SOT_THT:TO-92_Inline, symbol Transistor_BJT:S8550
- added R1, R10, R11, R12, R2, R21, R22, R23, R24, R3, R4, R9: 5.1k, symbol Device:R
- J1: renamed from J?; footprint (none) -> Connector_JST:JST_AUH_BM05B-AUHKS-GA-TB_1x05-1MP_P1.50mm_Vertical
- gave numbers to parts that had none: 19
Connections:
- net 5V: now also Q1.1 (E), Q2.1 (E), Q3.1 (E), Q4.1 (E), Q5.1 (E), Q6.1 (E), Q7.1 (E), Q8.1 (E), R1.1, R2.1, R3.1, R4.1
- net GND: now also R10.2, R11.2, R12.2, R21.2, R22.2, R23.2, R24.2, R9.2
- net GNDL: no longer U2.2, U2.4, U2.6, U2.8
- net Out1: now also Q1.3 (C), R12.1
- net Out2: now also Q2.3 (C), R11.1
- net Out3: now also Q3.3 (C), R10.1
- net Out4: now also Q4.3 (C), R9.1
- net Out5: now also Q5.3 (C), R24.1
- net Out6: now also Q6.3 (C), R23.1
- net Out7: now also Q7.3 (C), R22.1
- net Out8: now also Q8.3 (C), R21.1
- net at R13.2, U2.16: now also Q5.2 (B)
- net at R14.2, U2.14: now also Q6.2 (B)
- net at U1.12: now also Q3.2 (B), R3.2
- net at R16.2, U2.10: now also Q8.2 (B)
- net at R15.2, U2.12: now also Q7.2 (B)
- net at U1.10: now also Q4.2 (B), R4.2
- net at U1.14: now also Q2.2 (B), R2.2
- net at U1.16: now also Q1.2 (B), R1.2
- new net: U2.2, U2.4, U2.6, U2.8
Other:
- note added: "Revisar si esa huella de JST es la correcta"
- moved on the sheet: R13, R14, R15, R16, R17, R18, R19, R20, R5, R6, R7, R8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

Commit message: Push mid :V
Parts:
- Q1, Q2, Q3, Q4, Q5, Q6, Q7, Q8: footprint Package_TO_SOT_THT:TO-92_Inline -> Package_TO_SOT_SMD:TSOT-23
- U3, U4: footprint (none) -> Package_SO:SOIC-16_4.55x10.3mm_P1.27mm

Commit message: auxilio
Parts:
- removed Q1, Q2, Q3, Q4, Q5, Q6, Q7, Q8: S8550, Package_TO_SOT_SMD:TSOT-23, symbol Transistor_BJT:S8550
- removed R1, R10, R11, R12, R2, R21, R22, R23, R24, R3, R4, R9: 5.1k, symbol Device:R
- added Q? (x8): S8050, Package_TO_SOT_THT:TO-92_Inline, symbol Transistor_BJT:S8050
- added R? (x12): 5.1k, symbol Device:R
- J?: renamed from J1; footprint Connector_JST:JST_AUH_BM05B-AUHKS-GA-TB_1x05-1MP_P1.50mm_Vertical -> (none)
- U?: renamed from U4; footprint Package_SO:SOIC-16_4.55x10.3mm_P1.27mm -> (none)
- U?: renamed from U3; footprint Package_SO:SOIC-16_4.55x10.3mm_P1.27mm -> (none)
- renumbered C2 to C?, C1 to C?, J2 to J?, R20 to R?, R13 to R?, R16 to R?, R18 to R?, R15 to R?, R14 to R?, R8 to R?, R19 to R?, R6 to R?, R5 to R?, R7 to R?, R17 to R?, U2 to U?, U1 to U?
Connections:
- net 5V: now also R?.1, R?.1, R?.1, R?.1, R?.1, R?.1, R?.1, R?.1, R?.1, R?.1, R?.1, R?.1
- net GND: now also Q?.1 (E), Q?.1 (E), Q?.1 (E), Q?.1 (E), Q?.1 (E), Q?.1 (E), Q?.1 (E), Q?.1 (E)
- net GNDL: now also U?.2, U?.4, U?.6, U?.8
- net Out1: now also Q?.3 (C), R?.2
- net Out2: now also Q?.3 (C), R?.2
- net Out3: now also Q?.3 (C), R?.2
- net Out4: now also Q?.3 (C), R?.2
- net Out5: now also Q?.3 (C), R?.2
- net Out6: now also Q?.3 (C), R?.2
- net Out7: now also Q?.3 (C), R?.2
- net Out8: now also Q?.3 (C), R?.2
- net at R?.2, U?.16: now also Q?.2 (B)
- net at U?.12: now also Q?.2 (B), R?.2
- net at R?.2, U?.14: now also Q?.2 (B)
- net at R?.2, U?.10: now also Q?.2 (B)
- net at R?.2, U?.12: now also Q?.2 (B)
- net at U?.10: now also Q?.2 (B), R?.2
- net at U?.14: now also Q?.2 (B), R?.2
- net at U?.16: now also Q?.2 (B), R?.2
Other:
- note removed: "Revisar si esa huella de JST es la correcta"
- moved on the sheet: R?, U?A

Commit message: Support
Parts:
- removed Q? (x8): S8050, Package_TO_SOT_THT:TO-92_Inline, symbol Transistor_BJT:S8050
- removed R? (x12): 5.1k, symbol Device:R
- added Q1, Q2, Q3, Q4, Q5, Q6, Q7, Q8: S8550, Package_TO_SOT_SMD:TSOT-23, symbol Transistor_BJT:S8550
- added R1, R10, R11, R12, R2, R21, R22, R23, R24, R3, R4, R9: 5.1k, symbol Device:R
- J1: renamed from J?; footprint (none) -> Connector_JST:JST_AUH_BM05B-AUHKS-GA-TB_1x05-1MP_P1.50mm_Vertical
- U3, U4: renamed from U?; footprint (none) -> Package_SO:SOIC-16_4.55x10.3mm_P1.27mm
- gave numbers to parts that had none: 17
Connections:
- net 5V: now also Q1.1 (E), Q2.1 (E), Q3.1 (E), Q4.1 (E), Q5.1 (E), Q6.1 (E), Q7.1 (E), Q8.1 (E), R1.1, R2.1, R3.1, R4.1
- net GND: now also R10.2, R11.2, R12.2, R21.2, R22.2, R23.2, R24.2, R9.2
- net GNDL: no longer U2.2, U2.4, U2.6, U2.8
- net Out1: now also Q1.3 (C), R12.1
- net Out2: now also Q2.3 (C), R11.1
- net Out3: now also Q3.3 (C), R10.1
- net Out4: now also Q4.3 (C), R9.1
- net Out5: now also Q5.3 (C), R24.1
- net Out6: now also Q6.3 (C), R23.1
- net Out7: now also Q7.3 (C), R22.1
- net Out8: now also Q8.3 (C), R21.1
- net at R13.2, U2.16: now also Q5.2 (B)
- net at R14.2, U2.14: now also Q6.2 (B)
- net at U1.12: now also Q3.2 (B), R3.2
- net at R16.2, U2.10: now also Q8.2 (B)
- net at R15.2, U2.12: now also Q7.2 (B)
- net at U1.10: now also Q4.2 (B), R4.2
- net at U1.14: now also Q2.2 (B), R2.2
- net at U1.16: now also Q1.2 (B), R1.2
- new net: U2.2, U2.4, U2.6, U2.8
Other:
- note added: "Revisar si esa huella de JST es la correcta"
- moved on the sheet: R13, R14, R15, R16, R17, R18, R19, R20, R5, R6, R7, R8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

Commit message: Algunas huellas añadidas
Parts:
- J2: footprint (none) -> Connector_JST:JST_AUH_BM05B-AUHKS-GA-TB_1x05-1MP_P1.50mm_Vertical
Changed lines of the file:
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@@
       (effects (font (size 1.27 1.27)) (justify left))
     )
-    (property "Footprint" "" (id 2) (at 229.87 115.57 0)
+    (property "Footprint" "Connector_JST:JST_AUH_BM05B-AUHKS-GA-TB_1x05-1MP_P1.50mm_Vertical" (id 2) (at 229.87 115.57 0)
       (effects (font (size 1.27 1.27)) hide)
     )

Commit message: Eliminando el error de autosave
Parts:
- R1, R10, R11, R12, R13, R14, R15, R16, R17, R18, R19, R2, R20, R21, R22, R23, R24, R3, R4, R5, R6, R7, R8, R9: footprint (none) -> Resistor_SMD:R_1206_3216Metric_Pad1.30x1.75mm_HandSolder
Changed lines of the file:
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@@
     (property "Reference" "R20" (id 0) (at 49.53 133.35 90))
     (property "Value" "220" (id 1) (at 49.53 135.89 90))
-    (property "Footprint" "" (id 2) (at 49.53 140.208 90)
+    (property "Footprint" "Resistor_SMD:R_1206_3216Metric_Pad1.30x1.75mm_HandSolder" (id 2) (at 49.53 140.208 90)
       (effects (font (size 1.27 1.27)) hide)
     )
@@
       (effects (font (size 1.27 1.27)) (justify left))
     )
-    (property "Footprint" "" (id 2) (at 134.112 110.49 90)
+    (property "Footprint" "Resistor_SMD:R_1206_3216Metric_Pad1.30x1.75mm_HandSolder" (id 2) (at 134.112 110.49 90)
       (effects (font (size 1.27 1.27)) hide)
     )
@@
       (effects (font (size 1.27 1.27)) (justify left))
     )
-    (property "Footprint" "" (id 2) (at 98.552 40.64 90)
+    (property "Footprint" "Resistor_SMD:R_1206_3216Metric_Pad1.30x1.75mm_HandSolder" (id 2) (at 98.552 40.64 90)
       (effects (font (size 1.27 1.27)) hide)
     )
@@
       (effects (font (size 1.27 1.27)) (justify left))
     )
-    (property "Footprint" "" (id 2) (at 80.772 110.49 90)
+    (property "Footprint" "Resistor_SMD:R_1206_3216Metric_Pad1.30x1.75mm_HandSolder" (id 2) (at 80.772 110.49 90)
       (effects (font (size 1.27 1.27)) hide)
     )
@@
     (property "Reference" "R18" (id 0) (at 49.53 118.11 90))
     (property "Value" "220" (id 1) (at 49.53 120.65 90))
-    (property "Footprint" "" (id 2) (at 49.53 124.968 90)
+    (property "Footprint" "Resistor_SMD:R_1206_3216Metric_Pad1.30x1.75mm_HandSolder" (id 2) (at 49.53 124.968 90)
       (effects (font (size 1.27 1.27)) hide)
     )
@@
       (effects (font (size 1.27 1.27)) (justify left))
     )
-    (property "Footprint" "" (id 2) (at 107.442 80.01 90)
+    (property "Footprint" "Resistor_SMD:R_1206_3216Metric_Pad1.30x1.75mm_HandSolder" (id 2) (at 107.442 80.01 90)
       (effects (font (size 1.27 1.27)) hide)
     )
@@
       (effects (font (size 1.27 1.27)) (justify left))
     )
-    (property "Footprint" "" (id 2) (at 89.662 149.86 90)
+    (property "Footprint" "Resistor_SMD:R_1206_3216Metric_Pad1.30x1.75mm_HandSolder" (id 2) (at 89.662 149.86 90)
       (effects (font (size 1.27 1.27)) hide)
     )
@@
       (effects (font (size 1.27 1.27)) (justify left))
     )
-    (property "Footprint" "" (id 2) (at 134.112 40.64 90)
+    (property "Footprint" "Resistor_SMD:R_1206_3216Metric_Pad1.30x1.75mm_HandSolder" (id 2) (at 134.112 40.64 90)
       (effects (font (size 1.27 1.27)) hide)
     )
@@
       (effects (font (size 1.27 1.27)) (justify left))
     )
-    (property "Footprint" "" (id 2) (at 125.222 149.86 90)
+    (property "Footprint" "Resistor_SMD:R_1206_3216Metric_Pad1.30x1.75mm_HandSolder" (id 2) (at 125.222 149.86 90)
       (effects (font (size 1.27 1.27)) hide)
     )
@@
       (effects (font (size 1.27 1.27)) (justify left))
     )
-    (property "Footprint" "" (id 2) (at 143.002 80.01 90)
+    (property "Footprint" "Resistor_SMD:R_1206_3216Metric_Pad1.30x1.75mm_HandSolder" (id 2) (at 143.002 80.01 90)
       (effects (font (size 1.27 1.27)) hide)
     )
@@
       (effects (font (size 1.27 1.27)) (justify left))
     )
-    (property "Footprint" "" (id 2) (at 98.552 110.49 90)
+    (property "Footprint" "Resistor_SMD:R_1206_3216Metric_Pad1.30x1.75mm_HandSolder" (id 2) (at 98.552 110.49 90)
       (effects (font (size 1.27 1.27)) hide)
     )
@@
       (effects (font (size 1.27 1.27)) (justify left))
     )
-    (property "Footprint" "" (id 2) (at 107.442 149.86 90)
+    (property "Footprint" "Resistor_SMD:R_1206_3216Metric_Pad1.30x1.75mm_HandSolder" (id 2) (at 107.442 149.86 90)
       (effects (font (size 1.27 1.27)) hide)
     )
@@
       (effects (font (size 1.27 1.27)) (justify left))
     )
-    (property "Footprint" "" (id 2) (at 80.772 40.64 90)
+    (property "Footprint" "Resistor_SMD:R_1206_3216Metric_Pad1.30x1.75mm_HandSolder" (id 2) (at 80.772 40.64 90)
       (effects (font (size 1.27 1.27)) hide)
     )
@@
       (effects (font (size 1.27 1.27)) (justify left))
     )
-    (property "Footprint" "" (id 2) (at 143.002 149.86 90)
+    (property "Footprint" "Resistor_SMD:R_1206_3216Metric_Pad1.30x1.75mm_HandSolder" (id 2) (at 143.002 149.86 90)
       (effects (font (size 1.27 1.27)) hide)
     )
@@
       (effects (font (size 1.27 1.27)) (justify left))
     )
-    (property "Footprint" "" (id 2) (at 116.332 110.49 90)
+    (property "Footprint" "Resistor_SMD:R_1206_3216Metric_Pad1.30x1.75mm_HandSolder" (id 2) (at 116.332 110.49 90)
       (effects (font (size 1.27 1.27)) hide)
     )
@@
       (effects (font (size 1.27 1.27)) (justify left))
     )
-    (property "Footprint" "" (id 2) (at 116.332 40.64 90)
+    (property "Footprint" "Resistor_SMD:R_1206_3216Metric_Pad1.30x1.75mm_HandSolder" (id 2) (at 116.332 40.64 90)
       (effects (font (size 1.27 1.27)) hide)
     )
@@
       (effects (font (size 1.27 1.27)) (justify left))
     )
-    (property "Footprint" "" (id 2) (at 89.662 80.01 90)
+    (property "Footprint" "Resistor_SMD:R_1206_3216Metric_Pad1.30x1.75mm_HandSolder" (id 2) (at 89.662 80.01 90)
       (effects (font (size 1.27 1.27)) hide)
     )
@@
     (property "Reference" "R8" (id 0) (at 49.53 63.5 90))
     (property "Value" "220" (id 1) (at 49.53 66.04 90))
-    (property "Footprint" "" (id 2) (at 49.53 70.358 90)
+    (property "Footprint" "Resistor_SMD:R_1206_3216Metric_Pad1.30x1.75mm_HandSolder" (id 2) (at 49.53 70.358 90)
       (effects (font (size 1.27 1.27)) hide)
     )
@@
     (property "Reference" "R19" (id 0) (at 49.53 125.73 90))
     (property "Value" "220" (id 1) (at 49.53 128.27 90))
-    (property "Footprint" "" (id 2) (at 49.53 132.588 90)
+    (property "Footprint" "Resistor_SMD:R_1206_3216Metric_Pad1.30x1.75mm_HandSolder" (id 2) (at 49.53 132.588 90)
       (effects (font (size 1.27 1.27)) hide)
     )
@@
     (property "Reference" "R6" (id 0) (at 49.53 48.26 90))
     (property "Value" "220" (id 1) (at 49.53 50.8 90))
-    (property "Footprint" "" (id 2) (at 49.53 55.118 90)
+    (property "Footprint" "Resistor_SMD:R_1206_3216Metric_Pad1.30x1.75mm_HandSolder" (id 2) (at 49.53 55.118 90)
       (effects (font (size 1.27 1.27)) hide)
     )
@@
     (property "Reference" "R5" (id 0) (at 49.53 40.64 90))
     (property "Value" "220" (id 1) (at 49.53 43.18 90))
-    (property "Footprint" "" (id 2) (at 49.53 47.498 90)
+    (property "Footprint" "Resistor_SMD:R_1206_3216Metric_Pad1.30x1.75mm_HandSolder" (id 2) (at 49.53 47.498 90)
       (effects (font (size 1.27 1.27)) hide)
     )
@@
     (property "Reference" "R7" (id 0) (at 49.53 55.88 90))
     (property "Value" "220" (id 1) (at 49.53 58.42 90))
-    (property "Footprint" "" (id 2) (at 49.53 62.738 90)
+    (property "Footprint" "Resistor_SMD:R_1206_3216Metric_Pad1.30x1.75mm_HandSolder" (id 2) (at 49.53 62.738 90)
       (effects (font (size 1.27 1.27)) hide)
     )
@@
       (effects (font (size 1.27 1.27)) (justify left))
     )
-    (property "Footprint" "" (id 2) (at 125.222 80.01 90)
+    (property "Footprint" "Resistor_SMD:R_1206_3216Metric_Pad1.30x1.75mm_HandSolder" (id 2) (at 125.222 80.01 90)
       (effects (font (size 1.27 1.27)) hide)
     )
@@
     (property "Reference" "R17" (id 0) (at 49.53 110.49 90))
     (property "Value" "220" (id 1) (at 49.53 113.03 90))
-    (property "Footprint" "" (id 2) (at 49.53 117.348 90)
-      (effects (font (size 1.27 1.27)) hide)
-    )
+    (property "Footprint" "Resistor_SMD:R_1206_3216Metric_Pad1.30x1.75mm_HandSolder" (id 2) (at 49.53 117.348 90)
+      (effects (font (size 1.27 1.27)) hide)
+    )

Commit message: Etiquetas globales para alimentación añadidas
Parts:
- C1, C2: footprint (none) -> Capacitor_SMD:C_0201_0603Metric_Pad0.64x0.40mm_HandSolder
Connections:
- net GNDL: now also U2.2, U2.4, U2.6, U2.8
- net 12V renamed +12V
- net 5V renamed +5V
Changed lines of the file:
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@@
   (junction (at 127 34.29) (diameter 0) (color 0 0 0 0)
   )
+  (junction (at 55.88 120.65) (diameter 0) (color 0 0 0 0)
+  )
   (junction (at 73.66 58.42) (diameter 0) (color 0 0 0 0)
   )
@@
   (junction (at 144.78 85.09) (diameter 0) (color 0 0 0 0)
   )
+  (junction (at 55.88 99.06) (diameter 0) (color 0 0 0 0)
+  )
   (junction (at 135.89 45.72) (diameter 0) (color 0 0 0 0)
   )
@@
   )
   (wire (pts (xy 91.44 73.66) (xy 91.44 74.93))
+    (stroke (width 0) (type default) (color 0 0 0 0))
+  )
+  (wire (pts (xy 55.88 99.06) (xy 55.88 120.65))
     (stroke (width 0) (type default) (color 0 0 0 0))
   )
@@
     (effects (font (size 1.27 1.27)) (justify right))
   )
-  (hierarchical_label "12V" (shape input) (at 224.79 46.99 90)
-    (effects (font (size 1.27 1.27)) (justify left))
-  )
   (hierarchical_label "In7" (shape input) (at 41.91 130.81 180)
     (effects (font (size 1.27 1.27)) (justify right))
   )
-  (hierarchical_label "5V" (shape input) (at 144.78 101.6 90)
-    (effects (font (size 1.27 1.27)) (justify left))
-  )
-  (hierarchical_label "5V" (shape input) (at 144.78 31.75 90)
-    (effects (font (size 1.27 1.27)) (justify left))
-  )
   (hierarchical_label "In8" (shape input) (at 41.91 138.43 180)
     (effects (font (size 1.27 1.27)) (justify right))
@@
   (hierarchical_label "In3" (shape input) (at 41.91 60.96 180)
     (effects (font (size 1.27 1.27)) (justify right))
-  )
-  (hierarchical_label "12V" (shape input) (at 224.79 92.71 90)
-    (effects (font (size 1.27 1.27)) (justify left))
   )
   (hierarchical_label "In6" (shape input) (at 41.91 123.19 180)
@@
     (property "Reference" "C2" (id 0) (at 233.68 100.33 90))
     (property "Value" "100n" (id 1) (at 233.68 102.87 90))
-    (property "Footprint" "" (id 2) (at 237.49 106.9848 0)
+    (property "Footprint" "Capacitor_SMD:C_0201_0603Metric_Pad0.64x0.40mm_HandSolder" (id 2) (at 237.49 106.9848 0)
       (effects (font (size 1.27 1.27)) hide)
     )
@@
     (property "Reference" "C1" (id 0) (at 233.68 54.61 90))
     (property "Value" "100n" (id 1) (at 233.68 57.15 90))
-    (property "Footprint" "" (id 2) (at 237.49 61.2648 0)
+    (property "Footprint" "Capacitor_SMD:C_0201_0603Metric_Pad0.64x0.40mm_HandSolder" (id 2) (at 237.49 61.2648 0)
       (effects (font (size 1.27 1.27)) hide)
     )
@@
     (pin "3")
   )
+  (symbol (lib_id "power:+5V") (at 144.78 101.6 0) (unit 1)
+    (in_bom yes) (on_board yes) (fields_autoplaced)
+    (property "Reference" "#PWR026" (id 0) (at 144.78 105.41 0)
+      (effects (font (size 1.27 1.27)) hide)
+    )
+    (property "Value" "+5V" (id 1) (at 144.78 96.52 0))
+    (property "Footprint" "" (id 2) (at 144.78 101.6 0)
+      (effects (font (size 1.27 1.27)) hide)
+    )
+    (property "Datasheet" "" (id 3) (at 144.78 101.6 0)
+      (effects (font (size 1.27 1.27)) hide)
+    )
+    (pin "1")
+  )
   (symbol (lib_id "Device:R") (at 127 149.86 0) (unit 1)
     (in_bom yes) (on_board yes) (fields_autoplaced)
@@
     (pin "1")
   )
+  (symbol (lib_id "power:+12V") (at 224.79 46.99 0) (unit 1)
+    (in_bom yes) (on_board yes) (fields_autoplaced)
+    (property "Reference" "#PWR027" (id 0) (at 224.79 50.8 0)
+      (effects (font (size 1.27 1.27)) hide)
+    )
+    (property "Value" "+12V" (id 1) (at 224.79 41.91 0))
+    (property "Footprint" "" (id 2) (at 224.79 46.99 0)
+      (effects (font (size 1.27 1.27)) hide)
+    )
+    (property "Datasheet" "" (id 3) (at 224.79 46.99 0)
+      (effects (font (size 1.27 1.27)) hide)
+    )
+    (pin "1")
+  )
   (symbol (lib_id "Device:R") (at 144.78 80.01 0) (unit 1)
     (in_bom yes) (on_board yes) (fields_autoplaced)
@@
     (pin "1")
     (pin "2")
+  )
+  (symbol (lib_id "power:+5V") (at 144.78 31.75 0) (unit 1)
+    (in_bom yes) (on_board yes) (fields_autoplaced)
+    (property "Reference" "#PWR025" (id 0) (at 144.78 35.56 0)
+      (effects (font (size 1.27 1.27)) hide)
+    )
+    (property "Value" "+5V" (id 1) (at 144.78 26.67 0))
+    (property "Footprint" "" (id 2) (at 144.78 31.75 0)
+      (effects (font (size 1.27 1.27)) hide)
+    )
+    (property "Datasheet" "" (id 3) (at 144.78 31.75 0)
+      (effects (font (size 1.27 1.27)) hide)
+    )
+    (pin "1")
   )
   (symbol (lib_id "Connector_Generic:Conn_01x04") (at 229.87 69.85 0) (unit 1)
@@
       (effects (font (size 1.27 1.27)) hide)
     )
+    (pin "1")
+  )
+  (symbol (lib_id "power:+12V") (at 224.79 92.71 0) (unit 1)
+    (in_bom yes) (on_board yes) (fields_autoplaced)
+    (property "Reference" "#PWR028" (id 0) (at 224.79 96.52 0)
+      (effects (font (size 1.27 1.27)) hide)
+    )
+    (property "Value" "+12V" (id 1) (at 224.79 87.63 0))
+    (property "Footprint" "" (id 2) (at 224.79 92.71 0)
+      (effects (font (size 1.27 1.27)) hide)
+    )
+    (property "Datasheet" "" (id 3) (at 224.79 92.71 0)
+      (effects (font (size 1.27 1.27)) hide)
+    )
