File: Esquemáticos/ESP32/Motores.kicad_sch (KiCad schematic)
At the start: 40 parts, among them J1 Conector para bobinas del mot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, J2 Conector para bobinas del mot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, Q1 S8550, Q2 S8550, Q3 S8550, Q4 S8550, Q5 S8550, Q6 S8550, Q7 S8550, Q8 S8550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

Commit message: Actualizadas las huellas de R y C
De acuerdo con la recomendación del profe, ahora todas son 0603.
Parts:
- C1, C2: footprint Capacitor_SMD:C_0201_0603Metric_Pad0.64x0.40mm_HandSolder -> Capacitor_SMD:C_0603_1608Metric_Pad1.08x0.95mm_HandSolder
- R1, R10, R11, R12, R13, R14, R15, R16, R17, R18, R19, R2, R20, R21, R22, R23, R24, R3, R4, R5, R6, R7, R8, R9: footprint Resistor_SMD:R_1206_3216Metric_Pad1.30x1.75mm_HandSolder -> Resistor_SMD:R_0603_1608Metric_Pad0.98x0.95mm_HandSolder
Changed lines of the file:
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@@
     (property "Reference" "R20" (id 0) (at 49.53 133.35 90))
     (property "Value" "220" (id 1) (at 49.53 135.89 90))
-    (property "Footprint" "Resistor_SMD:R_1206_3216Metric_Pad1.30x1.75mm_HandSolder" (id 2) (at 49.53 140.208 90)
+    (property "Footprint" "Resistor_SMD:R_0603_1608Metric_Pad0.98x0.95mm_HandSolder" (id 2) (at 49.53 140.208 90)
       (effects (font (size 1.27 1.27)) hide)
     )
@@
       (effects (font (size 1.27 1.27)) (justify left))
     )
-    (property "Footprint" "Resistor_SMD:R_1206_3216Metric_Pad1.30x1.75mm_HandSolder" (id 2) (at 134.112 110.49 90)
+    (property "Footprint" "Resistor_SMD:R_0603_1608Metric_Pad0.98x0.95mm_HandSolder" (id 2) (at 134.112 110.49 90)
       (effects (font (size 1.27 1.27)) hide)
     )
@@
       (effects (font (size 1.27 1.27)) (justify left))
     )
-    (property "Footprint" "Resistor_SMD:R_1206_3216Metric_Pad1.30x1.75mm_HandSolder" (id 2) (at 98.552 40.64 90)
+    (property "Footprint" "Resistor_SMD:R_0603_1608Metric_Pad0.98x0.95mm_HandSolder" (id 2) (at 98.552 40.64 90)
       (effects (font (size 1.27 1.27)) hide)
     )
@@
     (property "Reference" "C2" (id 0) (at 233.68 100.33 90))
     (property "Value" "100n" (id 1) (at 233.68 102.87 90))
-    (property "Footprint" "Capacitor_SMD:C_0201_0603Metric_Pad0.64x0.40mm_HandSolder" (id 2) (at 237.49 106.9848 0)
+    (property "Footprint" "Capacitor_SMD:C_0603_1608Metric_Pad1.08x0.95mm_HandSolder" (id 2) (at 237.49 106.9848 0)
       (effects (font (size 1.27 1.27)) hide)
     )
@@
       (effects (font (size 1.27 1.27)) (justify left))
     )
-    (property "Footprint" "Resistor_SMD:R_1206_3216Metric_Pad1.30x1.75mm_HandSolder" (id 2) (at 80.772 110.49 90)
+    (property "Footprint" "Resistor_SMD:R_0603_1608Metric_Pad0.98x0.95mm_HandSolder" (id 2) (at 80.772 110.49 90)
       (effects (font (size 1.27 1.27)) hide)
     )
@@
     (property "Reference" "R18" (id 0) (at 49.53 118.11 90))
     (property "Value" "220" (id 1) (at 49.53 120.65 90))
-    (property "Footprint" "Resistor_SMD:R_1206_3216Metric_Pad1.30x1.75mm_HandSolder" (id 2) (at 49.53 124.968 90)
+    (property "Footprint" "Resistor_SMD:R_0603_1608Metric_Pad0.98x0.95mm_HandSolder" (id 2) (at 49.53 124.968 90)
       (effects (font (size 1.27 1.27)) hide)
     )
@@
       (effects (font (size 1.27 1.27)) (justify left))
     )
-    (property "Footprint" "Resistor_SMD:R_1206_3216Metric_Pad1.30x1.75mm_HandSolder" (id 2) (at 107.442 80.01 90)
+    (property "Footprint" "Resistor_SMD:R_0603_1608Metric_Pad0.98x0.95mm_HandSolder" (id 2) (at 107.442 80.01 90)
       (effects (font (size 1.27 1.27)) hide)
     )
@@
     (property "Reference" "C1" (id 0) (at 233.68 54.61 90))
     (property "Value" "100n" (id 1) (at 233.68 57.15 90))
-    (property "Footprint" "Capacitor_SMD:C_0201_0603Metric_Pad0.64x0.40mm_HandSolder" (id 2) (at 237.49 61.2648 0)
+    (property "Footprint" "Capacitor_SMD:C_0603_1608Metric_Pad1.08x0.95mm_HandSolder" (id 2) (at 237.49 61.2648 0)
       (effects (font (size 1.27 1.27)) hide)
     )
@@
       (effects (font (size 1.27 1.27)) (justify left))
     )
-    (property "Footprint" "Resistor_SMD:R_1206_3216Metric_Pad1.30x1.75mm_HandSolder" (id 2) (at 89.662 149.86 90)
+    (property "Footprint" "Resistor_SMD:R_0603_1608Metric_Pad0.98x0.95mm_HandSolder" (id 2) (at 89.662 149.86 90)
       (effects (font (size 1.27 1.27)) hide)
     )
@@
       (effects (font (size 1.27 1.27)) (justify left))
     )
-    (property "Footprint" "Resistor_SMD:R_1206_3216Metric_Pad1.30x1.75mm_HandSolder" (id 2) (at 134.112 40.64 90)
+    (property "Footprint" "Resistor_SMD:R_0603_1608Metric_Pad0.98x0.95mm_HandSolder" (id 2) (at 134.112 40.64 90)
       (effects (font (size 1.27 1.27)) hide)
     )
@@
       (effects (font (size 1.27 1.27)) (justify left))
     )
-    (property "Footprint" "Resistor_SMD:R_1206_3216Metric_Pad1.30x1.75mm_HandSolder" (id 2) (at 125.222 149.86 90)
+    (property "Footprint" "Resistor_SMD:R_0603_1608Metric_Pad0.98x0.95mm_HandSolder" (id 2) (at 125.222 149.86 90)
       (effects (font (size 1.27 1.27)) hide)
     )
@@
       (effects (font (size 1.27 1.27)) (justify left))
     )
-    (property "Footprint" "Resistor_SMD:R_1206_3216Metric_Pad1.30x1.75mm_HandSolder" (id 2) (at 143.002 80.01 90)
+    (property "Footprint" "Resistor_SMD:R_0603_1608Metric_Pad0.98x0.95mm_HandSolder" (id 2) (at 143.002 80.01 90)
       (effects (font (size 1.27 1.27)) hide)
     )
@@
       (effects (font (size 1.27 1.27)) (justify left))
     )
-    (property "Footprint" "Resistor_SMD:R_1206_3216Metric_Pad1.30x1.75mm_HandSolder" (id 2) (at 98.552 110.49 90)
+    (property "Footprint" "Resistor_SMD:R_0603_1608Metric_Pad0.98x0.95mm_HandSolder" (id 2) (at 98.552 110.49 90)
       (effects (font (size 1.27 1.27)) hide)
     )
@@
       (effects (font (size 1.27 1.27)) (justify left))
     )
-    (property "Footprint" "Resistor_SMD:R_1206_3216Metric_Pad1.30x1.75mm_HandSolder" (id 2) (at 107.442 149.86 90)
+    (property "Footprint" "Resistor_SMD:R_0603_1608Metric_Pad0.98x0.95mm_HandSolder" (id 2) (at 107.442 149.86 90)
       (effects (font (size 1.27 1.27)) hide)
     )
@@
       (effects (font (size 1.27 1.27)) (justify left))
     )
-    (property "Footprint" "Resistor_SMD:R_1206_3216Metric_Pad1.30x1.75mm_HandSolder" (id 2) (at 80.772 40.64 90)
+    (property "Footprint" "Resistor_SMD:R_0603_1608Metric_Pad0.98x0.95mm_HandSolder" (id 2) (at 80.772 40.64 90)
       (effects (font (size 1.27 1.27)) hide)
     )
@@
       (effects (font (size 1.27 1.27)) (justify left))
     )
-    (property "Footprint" "Resistor_SMD:R_1206_3216Metric_Pad1.30x1.75mm_HandSolder" (id 2) (at 143.002 149.86 90)
+    (property "Footprint" "Resistor_SMD:R_0603_1608Metric_Pad0.98x0.95mm_HandSolder" (id 2) (at 143.002 149.86 90)
       (effects (font (size 1.27 1.27)) hide)
     )
@@
       (effects (font (size 1.27 1.27)) (justify left))
     )
-    (property "Footprint" "Resistor_SMD:R_1206_3216Metric_Pad1.30x1.75mm_HandSolder" (id 2) (at 116.332 110.49 90)
+    (property "Footprint" "Resistor_SMD:R_0603_1608Metric_Pad0.98x0.95mm_HandSolder" (id 2) (at 116.332 110.49 90)
       (effects (font (size 1.27 1.27)) hide)
     )
@@
       (effects (font (size 1.27 1.27)) (justify left))
     )
-    (property "Footprint" "Resistor_SMD:R_1206_3216Metric_Pad1.30x1.75mm_HandSolder" (id 2) (at 116.332 40.64 90)
+    (property "Footprint" "Resistor_SMD:R_0603_1608Metric_Pad0.98x0.95mm_HandSolder" (id 2) (at 116.332 40.64 90)
       (effects (font (size 1.27 1.27)) hide)
     )
@@
       (effects (font (size 1.27 1.27)) (justify left))
     )
-    (property "Footprint" "Resistor_SMD:R_1206_3216Metric_Pad1.30x1.75mm_HandSolder" (id 2) (at 89.662 80.01 90)
+    (property "Footprint" "Resistor_SMD:R_0603_1608Metric_Pad0.98x0.95mm_HandSolder" (id 2) (at 89.662 80.01 90)
       (effects (font (size 1.27 1.27)) hide)
     )
@@
     (property "Reference" "R8" (id 0) (at 49.53 63.5 90))
     (property "Value" "220" (id 1) (at 49.53 66.04 90))
-    (property "Footprint" "Resistor_SMD:R_1206_3216Metric_Pad1.30x1.75mm_HandSolder" (id 2) (at 49.53 70.358 90)
+    (property "Footprint" "Resistor_SMD:R_0603_1608Metric_Pad0.98x0.95mm_HandSolder" (id 2) (at 49.53 70.358 90)
       (effects (font (size 1.27 1.27)) hide)
     )
@@
     (property "Reference" "R19" (id 0) (at 49.53 125.73 90))
     (property "Value" "220" (id 1) (at 49.53 128.27 90))
-    (property "Footprint" "Resistor_SMD:R_1206_3216Metric_Pad1.30x1.75mm_HandSolder" (id 2) (at 49.53 132.588 90)
+    (property "Footprint" "Resistor_SMD:R_0603_1608Metric_Pad0.98x0.95mm_HandSolder" (id 2) (at 49.53 132.588 90)
       (effects (font (size 1.27 1.27)) hide)
     )
@@
     (property "Reference" "R6" (id 0) (at 49.53 48.26 90))
     (property "Value" "220" (id 1) (at 49.53 50.8 90))
-    (property "Footprint" "Resistor_SMD:R_1206_3216Metric_Pad1.30x1.75mm_HandSolder" (id 2) (at 49.53 55.118 90)
+    (property "Footprint" "Resistor_SMD:R_0603_1608Metric_Pad0.98x0.95mm_HandSolder" (id 2) (at 49.53 55.118 90)
       (effects (font (size 1.27 1.27)) hide)
     )
@@
     (property "Reference" "R5" (id 0) (at 49.53 40.64 90))
     (property "Value" "220" (id 1) (at 49.53 43.18 90))
-    (property "Footprint" "Resistor_SMD:R_1206_3216Metric_Pad1.30x1.75mm_HandSolder" (id 2) (at 49.53 47.498 90)
+    (property "Footprint" "Resistor_SMD:R_0603_1608Metric_Pad0.98x0.95mm_HandSolder" (id 2) (at 49.53 47.498 90)
       (effects (font (size 1.27 1.27)) hide)
     )
@@
     (property "Reference" "R7" (id 0) (at 49.53 55.88 90))
     (property "Value" "220" (id 1) (at 49.53 58.42 90))
-    (property "Footprint" "Resistor_SMD:R_1206_3216Metric_Pad1.30x1.75mm_HandSolder" (id 2) (at 49.53 62.738 90)
+    (property "Footprint" "Resistor_SMD:R_0603_1608Metric_Pad0.98x0.95mm_HandSolder" (id 2) (at 49.53 62.738 90)
       (effects (font (size 1.27 1.27)) hide)
     )
@@
       (effects (font (size 1.27 1.27)) (justify left))
     )
-    (property "Footprint" "Resistor_SMD:R_1206_3216Metric_Pad1.30x1.75mm_HandSolder" (id 2) (at 125.222 80.01 90)
+    (property "Footprint" "Resistor_SMD:R_0603_1608Metric_Pad0.98x0.95mm_HandSolder" (id 2) (at 125.222 80.01 90)
       (effects (font (size 1.27 1.27)) hide)
     )
@@
     (property "Reference" "R17" (id 0) (at 49.53 110.49 90))
     (property "Value" "220" (id 1) (at 49.53 113.03 90))
-    (property "Footprint" "Resistor_SMD:R_1206_3216Metric_Pad1.30x1.75mm_HandSolder" (id 2) (at 49.53 117.348 90)
-      (effects (font (size 1.27 1.27)) hide)
-    )
+    (property "Footprint" "Resistor_SMD:R_0603_1608Metric_Pad0.98x0.95mm_HandSolder" (id 2) (at 49.53 117.348 90)
+      (effects (font (size 1.27 1.27)) hide)
+    )

Commit message: PCB versión 1 (Faltan zonas de GND)
Parts:
- J1, J2: footprint Connector_JST:JST_AUH_BM05B-AUHKS-GA-TB_1x05-1MP_P1.50mm_Vertical -> Connector_JST:JST_EH_B5B-EH-A_1x05_P2.50mm_Vertical; symbol Connector_Generic:Conn_01x04 -> Connector_Generic:Conn_01x05
Connections:
- net +12V: now also J1.1 (Pin_1), J2.1 (Pin_1)
- net at U4.13 (O4): now also J2.5 (Pin_5); no longer J2.4 (Pin_4)
- net at U4.14 (O3): now also J2.4 (Pin_4); no longer J2.3 (Pin_3)
- net at U4.15 (O2): now also J2.3 (Pin_3); no longer J2.2 (Pin_2)
- net at U4.16 (O1): now also J2.2 (Pin_2); no longer J2.1 (Pin_1)
- net at U3.13 (O4): now also J1.5 (Pin_5); no longer J1.4 (Pin_4)
- net at U3.14 (O3): now also J1.4 (Pin_4); no longer J1.3 (Pin_3)
- net at U3.15 (O2): now also J1.3 (Pin_3); no longer J1.2 (Pin_2)
- net at U3.16 (O1): now also J1.2 (Pin_2); no longer J1.1 (Pin_1)
Other:
- note removed: "Revisar si esa huella de JST es la correcta"
Changed lines of the file:
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@@
-    (stroke (width 0) (type default) (color 0 0 0 0))
-  )
-  (polyline (pts (xy 233.68 77.47) (xy 233.68 83.82))
     (stroke (width 0) (type default) (color 0 0 0 0))
   )
@@
     (stroke (width 0) (type default) (color 0 0 0 0))
   )
-  (polyline (pts (xy 233.68 83.82) (xy 259.08 83.82))
-    (stroke (width 0) (type default) (color 0 0 0 0))
-  )
   (wire (pts (xy 91.44 104.14) (xy 91.44 133.35))
     (stroke (width 0) (type default) (color 0 0 0 0))
@@
     (stroke (width 0) (type default) (color 0 0 0 0))
   )
+  (wire (pts (xy 224.79 107.95) (xy 224.79 110.49))
+    (stroke (width 0) (type default) (color 0 0 0 0))
+  )
   (wire (pts (xy 109.22 34.29) (xy 118.11 34.29))
     (stroke (width 0) (type default) (color 0 0 0 0))
@@
   )
   (wire (pts (xy 82.55 36.83) (xy 82.55 34.29))
+    (stroke (width 0) (type default) (color 0 0 0 0))
+  )
+  (wire (pts (xy 224.79 62.23) (xy 224.79 64.77))
     (stroke (width 0) (type default) (color 0 0 0 0))
   )
@@
   (text "Revisar bien si esto es correcto (Meter 12V alegremente)"
     (at 85.09 29.21 0)
-    (effects (font (size 1.27 1.27)) (justify left bottom))
-  )
-  (text "Revisar si esa huella de\nJST es la correcta" (at 234.95 82.55 0)
     (effects (font (size 1.27 1.27)) (justify left bottom))
   )
@@
     (pin "1")
   )
-  (symbol (lib_id "Connector_Generic:Conn_01x04") (at 229.87 69.85 0) (unit 1)
+  (symbol (lib_id "Connector_Generic:Conn_01x05") (at 229.87 69.85 0) (unit 1)
     (in_bom yes) (on_board yes) (fields_autoplaced)
     (property "Reference" "J1" (id 0) (at 232.41 69.8499 0)
@@
       (effects (font (size 1.27 1.27)) (justify left))
     )
-    (property "Footprint" "Connector_JST:JST_AUH_BM05B-AUHKS-GA-TB_1x05-1MP_P1.50mm_Vertical" (id 2) (at 229.87 69.85 0)
+    (property "Footprint" "Connector_JST:JST_EH_B5B-EH-A_1x05_P2.50mm_Vertical" (id 2) (at 229.87 69.85 0)
       (effects (font (size 1.27 1.27)) hide)
     )
@@
     (pin "3")
     (pin "4")
+    (pin "5")
   )
   (symbol (lib_id "Transistor_BJT:S8550") (at 106.68 60.96 0) (mirror x) (unit 1)
@@
     (pin "3")
   )
-  (symbol (lib_id "Connector_Generic:Conn_01x04") (at 229.87 115.57 0) (unit 1)
+  (symbol (lib_id "Connector_Generic:Conn_01x05") (at 229.87 115.57 0) (unit 1)
     (in_bom yes) (on_board yes) (fields_autoplaced)
     (property "Reference" "J2" (id 0) (at 232.41 115.5699 0)
@@
       (effects (font (size 1.27 1.27)) (justify left))
     )
-    (property "Footprint" "Connector_JST:JST_AUH_BM05B-AUHKS-GA-TB_1x05-1MP_P1.50mm_Vertical" (id 2) (at 229.87 115.57 0)
+    (property "Footprint" "Connector_JST:JST_EH_B5B-EH-A_1x05_P2.50mm_Vertical" (id 2) (at 229.87 115.57 0)
       (effects (font (size 1.27 1.27)) hide)
     )
@@
     (pin "3")
     (pin "4")
+    (pin "5")
   )
   (symbol (lib_id "Device:R") (at 91.44 80.01 0) (unit 1)

Commit message: Añadí las conexiones con los optoacopladores
Además arreglé la posición de algunas vías.
Connections:
- net GNDL is gone; now on net GND: U1.2, U1.4, U1.6, U1.8, U2.2, U2.4, U2.6, U2.8
Changed lines of the file:
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@@
   (junction (at 100.33 130.81) (diameter 0) (color 0 0 0 0)
   )
+  (junction (at 55.88 143.51) (diameter 0) (color 0 0 0 0)
+  )
   (junction (at 127 34.29) (diameter 0) (color 0 0 0 0)
   )
-  (junction (at 55.88 120.65) (diameter 0) (color 0 0 0 0)
-  )
   (junction (at 73.66 58.42) (diameter 0) (color 0 0 0 0)
   )
@@
   (junction (at 55.88 66.04) (diameter 0) (color 0 0 0 0)
   )
+  (junction (at 55.88 73.66) (diameter 0) (color 0 0 0 0)
+  )
   (junction (at 82.55 138.43) (diameter 0) (color 0 0 0 0)
   )
@@
   (junction (at 144.78 85.09) (diameter 0) (color 0 0 0 0)
   )
-  (junction (at 55.88 99.06) (diameter 0) (color 0 0 0 0)
-  )
   (junction (at 135.89 45.72) (diameter 0) (color 0 0 0 0)
   )
@@
   (junction (at 91.44 85.09) (diameter 0) (color 0 0 0 0)
   )
-  (junction (at 55.88 73.66) (diameter 0) (color 0 0 0 0)
-  )
   (junction (at 109.22 34.29) (diameter 0) (color 0 0 0 0)
   )
@@
     (stroke (width 0) (type default) (color 0 0 0 0))
   )
-  (wire (pts (xy 55.88 99.06) (xy 55.88 120.65))
-    (stroke (width 0) (type default) (color 0 0 0 0))
-  )
   (wire (pts (xy 190.5 67.31) (xy 199.39 67.31))
     (stroke (width 0) (type default) (color 0 0 0 0))
@@
     (stroke (width 0) (type default) (color 0 0 0 0))
   )
-  (wire (pts (xy 55.88 73.66) (xy 55.88 99.06))
-    (stroke (width 0) (type default) (color 0 0 0 0))
-  )
   (polyline (pts (xy 181.61 147.32) (xy 270.51 147.32))
     (stroke (width 0) (type default) (color 0 0 0 0))
@@
     (stroke (width 0) (type default) (color 0 0 0 0))
   )
+  (wire (pts (xy 55.88 73.66) (xy 55.88 85.09))
+    (stroke (width 0) (type default) (color 0 0 0 0))
+  )
   (wire (pts (xy 144.78 85.09) (xy 144.78 88.9))
     (stroke (width 0) (type default) (color 0 0 0 0))
@@
     (stroke (width 0) (type default) (color 0 0 0 0))
   )
+  (wire (pts (xy 55.88 143.51) (xy 55.88 154.94))
+    (stroke (width 0) (type default) (color 0 0 0 0))
+  )
   (wire (pts (xy 82.55 36.83) (xy 82.55 34.29))
     (stroke (width 0) (type default) (color 0 0 0 0))
@@
   )
   (wire (pts (xy 72.39 138.43) (xy 82.55 138.43))
-    (stroke (width 0) (type default) (color 0 0 0 0))
-  )
-  (wire (pts (xy 41.91 99.06) (xy 55.88 99.06))
     (stroke (width 0) (type default) (color 0 0 0 0))
   )
@@
   )
   (hierarchical_label "In4" (shape input) (at 41.91 68.58 180)
-    (effects (font (size 1.27 1.27)) (justify right))
-  )
-  (hierarchical_label "GNDL" (shape input) (at 41.91 99.06 180)
     (effects (font (size 1.27 1.27)) (justify right))
   )
@@
     (pin "2")
   )
+  (symbol (lib_id "power:GND") (at 55.88 85.09 0) (unit 1)
+    (in_bom yes) (on_board yes) (fields_autoplaced)
+    (property "Reference" "#PWR?" (id 0) (at 55.88 91.44 0)
+      (effects (font (size 1.27 1.27)) hide)
+    )
+    (property "Value" "GND" (id 1) (at 55.88 90.17 0))
+    (property "Footprint" "" (id 2) (at 55.88 85.09 0)
+      (effects (font (size 1.27 1.27)) hide)
+    )
+    (property "Datasheet" "" (id 3) (at 55.88 85.09 0)
+      (effects (font (size 1.27 1.27)) hide)
+    )
+    (pin "1")
+  )
   (symbol (lib_id "Transistor_Array:ULN2003A") (at 209.55 72.39 0) (unit 1)
     (in_bom yes) (on_board yes) (fields_autoplaced)
@@
     (pin "5")
   )
+  (symbol (lib_id "power:GND") (at 55.88 154.94 0) (unit 1)
+    (in_bom yes) (on_board yes) (fields_autoplaced)
+    (property "Reference" "#PWR?" (id 0) (at 55.88 161.29 0)
+      (effects (font (size 1.27 1.27)) hide)
+    )
+    (property "Value" "GND" (id 1) (at 55.88 160.02 0))
+    (property "Footprint" "" (id 2) (at 55.88 154.94 0)
+      (effects (font (size 1.27 1.27)) hide)
+    )
+    (property "Datasheet" "" (id 3) (at 55.88 154.94 0)
+      (effects (font (size 1.27 1.27)) hide)
+    )
+    (pin "1")
+  )
   (symbol (lib_id "Device:R") (at 91.44 80.01 0) (unit 1)

Commit message: Huellas actualizadas según los vendedores locales
Falta la del optoacoplador y actualizar la placa. Además, dependiendo de la resñpuesta del profe tocaría re-diseñar todo :c
Parts:
- C1, C2: value 100n -> 0.1uF; footprint Capacitor_SMD:C_0603_1608Metric_Pad1.08x0.95mm_HandSolder -> Capacitor_SMD:C_0805_2012Metric_Pad1.18x1.45mm_HandSolder
- R1, R10, R11, R12, R13, R14, R15, R16, R17, R18, R19, R2, R20, R21, R22, R23, R24, R3, R4, R5, R6, R7, R8, R9: footprint Resistor_SMD:R_0603_1608Metric_Pad0.98x0.95mm_HandSolder -> Resistor_SMD:R_0805_2012Metric_Pad1.20x1.40mm_HandSolder
- U3, U4: footprint Package_SO:SOIC-16_4.55x10.3mm_P1.27mm -> Package_DIP:DIP-16_W7.62mm_Socket
Other:
- note removed: "Revisar bien si esto es correcto (Conectar a la tierra común acá)"
- note removed: "Revisar bien si esto es correcto (Meter 12V alegremente)"

Commit message: NewPCB
Parts:
- U1, U2: footprint Package_SO:SOP-16_4.4x10.4mm_P1.27mm -> Package_DIP:DIP-16_W7.62mm_Socket
Changed lines of the file:
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@@
     (property "Reference" "U2" (id 0) (at 64.77 109.22 0))
     (property "Value" "LTV-247" (id 1) (at 64.77 111.76 0))
-    (property "Footprint" "Package_SO:SOP-16_4.4x10.4mm_P1.27mm" (id 2) (at 59.69 123.19 0)
+    (property "Footprint" "Package_DIP:DIP-16_W7.62mm_Socket" (id 2) (at 59.69 123.19 0)
       (effects (font (size 1.27 1.27) italic) (justify left) hide)
     )
@@
       (effects (font (size 1.27 1.27)) hide)
     )
-    (property "Footprint" "Package_SO:SOP-16_4.4x10.4mm_P1.27mm" (id 2) (at 59.69 130.81 0)
+    (property "Footprint" "Package_DIP:DIP-16_W7.62mm_Socket" (id 2) (at 59.69 130.81 0)
       (effects (font (size 1.27 1.27) italic) (justify left) hide)
     )
@@
       (effects (font (size 1.27 1.27)) hide)
     )
-    (property "Footprint" "Package_SO:SOP-16_4.4x10.4mm_P1.27mm" (id 2) (at 59.69 68.58 0)
+    (property "Footprint" "Package_DIP:DIP-16_W7.62mm_Socket" (id 2) (at 59.69 68.58 0)
       (effects (font (size 1.27 1.27) italic) (justify left) hide)
     )
@@
       (effects (font (size 1.27 1.27)) hide)
     )
-    (property "Footprint" "Package_SO:SOP-16_4.4x10.4mm_P1.27mm" (id 2) (at 59.69 138.43 0)
+    (property "Footprint" "Package_DIP:DIP-16_W7.62mm_Socket" (id 2) (at 59.69 138.43 0)
       (effects (font (size 1.27 1.27) italic) (justify left) hide)
     )
@@
       (effects (font (size 1.27 1.27)) hide)
     )
-    (property "Footprint" "Package_SO:SOP-16_4.4x10.4mm_P1.27mm" (id 2) (at 59.69 76.2 0)
+    (property "Footprint" "Package_DIP:DIP-16_W7.62mm_Socket" (id 2) (at 59.69 76.2 0)
       (effects (font (size 1.27 1.27) italic) (justify left) hide)
     )
@@
       (effects (font (size 1.27 1.27)) hide)
     )
-    (property "Footprint" "Package_SO:SOP-16_4.4x10.4mm_P1.27mm" (id 2) (at 59.69 60.96 0)
+    (property "Footprint" "Package_DIP:DIP-16_W7.62mm_Socket" (id 2) (at 59.69 60.96 0)
       (effects (font (size 1.27 1.27) italic) (justify left) hide)
     )
@@
     (property "Reference" "U1" (id 0) (at 64.77 39.37 0))
     (property "Value" "LTV-247" (id 1) (at 64.77 41.91 0))
-    (property "Footprint" "Package_SO:SOP-16_4.4x10.4mm_P1.27mm" (id 2) (at 59.69 53.34 0)
+    (property "Footprint" "Package_DIP:DIP-16_W7.62mm_Socket" (id 2) (at 59.69 53.34 0)
       (effects (font (size 1.27 1.27) italic) (justify left) hide)
     )
@@
       (effects (font (size 1.27 1.27)) hide)
     )
-    (property "Footprint" "Package_SO:SOP-16_4.4x10.4mm_P1.27mm" (id 2) (at 59.69 146.05 0)
-      (effects (font (size 1.27 1.27) italic) (justify left) hide)
-    )
+    (property "Footprint" "Package_DIP:DIP-16_W7.62mm_Socket" (id 2) (at 59.69 146.05 0)
+      (effects (font (size 1.27 1.27) italic) (justify left) hide)
+    )
