File: Esquemáticos/ESP32/Motores.kicad_sch (KiCad schematic)
At the start: 40 parts, among them J1 Conector para bobinas del mot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, J2 Conector para bobinas del mot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, Q1 S8550, Q2 S8550, Q3 S8550, Q4 S8550, Q5 S8550, Q6 S8550, Q7 S8550, Q8 S8550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

Commit message: PCB terminada
Revisar los gerber y los drill :3
Connections:
- net +12V is gone; now on net +5V: C1.1, C2.1, J1.1 (Pin_1), J2.1 (Pin_1), U3.9 (COM), U4.9 (COM)
Changed lines of the file:
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@@
     (pin "9")
+  )
+  (symbol (lib_id "power:+5V") (at 224.79 92.71 0) (unit 1)
+    (in_bom yes) (on_board yes) (fields_autoplaced)
+    (property "Reference" "#PWR?" (id 0) (at 224.79 96.52 0)
+      (effects (font (size 1.27 1.27)) hide)
+    )
+    (property "Value" "+5V" (id 1) (at 224.79 87.63 0))
+    (property "Footprint" "" (id 2) (at 224.79 92.71 0)
+      (effects (font (size 1.27 1.27)) hide)
+    )
+    (property "Datasheet" "" (id 3) (at 224.79 92.71 0)
+      (effects (font (size 1.27 1.27)) hide)
+    )
+    (pin "1")
   )
   (symbol (lib_id "Device:R") (at 49.53 138.43 90) (unit 1)
@@
     (pin "1")
   )
-  (symbol (lib_id "power:+12V") (at 224.79 46.99 0) (unit 1)
-    (in_bom yes) (on_board yes) (fields_autoplaced)
-    (property "Reference" "#PWR027" (id 0) (at 224.79 50.8 0)
-      (effects (font (size 1.27 1.27)) hide)
-    )
-    (property "Value" "+12V" (id 1) (at 224.79 41.91 0))
+  (symbol (lib_id "power:+5V") (at 224.79 46.99 0) (unit 1)
+    (in_bom yes) (on_board yes) (fields_autoplaced)
+    (property "Reference" "#PWR?" (id 0) (at 224.79 50.8 0)
+      (effects (font (size 1.27 1.27)) hide)
+    )
+    (property "Value" "+5V" (id 1) (at 224.79 41.91 0))
     (property "Footprint" "" (id 2) (at 224.79 46.99 0)
       (effects (font (size 1.27 1.27)) hide)
@@
       (effects (font (size 1.27 1.27)) hide)
     )
-    (pin "1")
-  )
-  (symbol (lib_id "power:+12V") (at 224.79 92.71 0) (unit 1)
-    (in_bom yes) (on_board yes) (fields_autoplaced)
-    (property "Reference" "#PWR028" (id 0) (at 224.79 96.52 0)
-      (effects (font (size 1.27 1.27)) hide)
-    )
-    (property "Value" "+12V" (id 1) (at 224.79 87.63 0))
-    (property "Footprint" "" (id 2) (at 224.79 92.71 0)
-      (effects (font (size 1.27 1.27)) hide)
-    )
-    (property "Datasheet" "" (id 3) (at 224.79 92.71 0)
-      (effects (font (size 1.27 1.27)) hide)
-    )
