File: Esquemáticos/ESP32/Potencia.kicad_sch (KiCad schematic)
At the start: 16 parts, among them U1 LM2596S-5

Commit message: Cambios hechos al esquemático, faltan detalles
Revisar el discord para dejar todo al día con el feedback de hoy
Parts:
- removed J?: Barrel_Jack, symbol Connector:Barrel_Jack
- removed SW?: SW_DIP_x01, symbol Switch:SW_DIP_x01
- added J?: Barrel_Jack, symbol Connector:Barrel_Jack
- added SW?: SW_DIP_x01, symbol Switch:SW_DIP_x01
Connections:
- net 12V: now also C?.1, C?.1, D1.2 (A), U?.3 (VI), SW?.2; no longer C1.1, C2.1, D1.1 (K), U1.1 (VIN)
- net 5V: no longer C?.1, C?.1, U?.3 (VI)
- net Earth: now also J?.2
- new net: J?.1, SW?.1
- new net: C1.1, C2.1, D1.1 (K), U1.1 (VIN)
Other:
- note added: "Etapa de potencia"
Changed lines of the file:
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@@
   (junction (at 129.54 119.38) (diameter 0) (color 0 0 0 0)
   )
+  (junction (at 99.06 86.36) (diameter 0) (color 0 0 0 0)
+  )
   (junction (at 176.53 119.38) (diameter 0) (color 0 0 0 0)
   )
@@
   (junction (at 217.17 63.5) (diameter 0) (color 0 0 0 0)
   )
-  (wire (pts (xy 87.63 68.58) (xy 92.71 68.58))
-    (stroke (width 0) (type default) (color 0 0 0 0))
-  )
   (wire (pts (xy 193.04 134.62) (xy 176.53 134.62))
     (stroke (width 0) (type default) (color 0 0 0 0))
@@
     (stroke (width 0) (type default) (color 0 0 0 0))
   )
+  (wire (pts (xy 99.06 86.36) (xy 102.87 86.36))
+    (stroke (width 0) (type default) (color 0 0 0 0))
+  )
   (wire (pts (xy 158.75 68.58) (xy 158.75 82.55))
     (stroke (width 0) (type default) (color 0 0 0 0))
@@
     (stroke (width 0) (type default) (color 0 0 0 0))
   )
-  (wire (pts (xy 129.54 113.03) (xy 129.54 119.38))
+  (wire (pts (xy 121.92 119.38) (xy 129.54 119.38))
     (stroke (width 0) (type default) (color 0 0 0 0))
   )
@@
     (stroke (width 0) (type default) (color 0 0 0 0))
   )
-  (wire (pts (xy 142.24 57.15) (xy 142.24 63.5))
-    (stroke (width 0) (type default) (color 0 0 0 0))
-  )
   (wire (pts (xy 203.2 63.5) (xy 217.17 63.5))
     (stroke (width 0) (type default) (color 0 0 0 0))
@@
     (stroke (width 0) (type default) (color 0 0 0 0))
   )
-  (wire (pts (xy 87.63 63.5) (xy 95.25 63.5))
-    (stroke (width 0) (type default) (color 0 0 0 0))
-  )
   (wire (pts (xy 129.54 119.38) (xy 140.97 119.38))
     (stroke (width 0) (type default) (color 0 0 0 0))
   )
-  (wire (pts (xy 92.71 68.58) (xy 92.71 82.55))
+  (wire (pts (xy 72.39 91.44) (xy 77.47 91.44))
+    (stroke (width 0) (type default) (color 0 0 0 0))
+  )
+  (wire (pts (xy 217.17 63.5) (xy 226.06 63.5))
     (stroke (width 0) (type default) (color 0 0 0 0))
   )
@@
     (stroke (width 0) (type default) (color 0 0 0 0))
   )
+  (wire (pts (xy 72.39 86.36) (xy 80.01 86.36))
+    (stroke (width 0) (type default) (color 0 0 0 0))
+  )
   (wire (pts (xy 176.53 119.38) (xy 176.53 121.92))
     (stroke (width 0) (type default) (color 0 0 0 0))
   )
+  (wire (pts (xy 99.06 81.28) (xy 99.06 86.36))
+    (stroke (width 0) (type default) (color 0 0 0 0))
+  )
   (wire (pts (xy 212.09 68.58) (xy 217.17 68.58))
     (stroke (width 0) (type default) (color 0 0 0 0))
@@
     (stroke (width 0) (type default) (color 0 0 0 0))
   )
+  (wire (pts (xy 95.25 86.36) (xy 99.06 86.36))
+    (stroke (width 0) (type default) (color 0 0 0 0))
+  )
   (wire (pts (xy 176.53 119.38) (xy 193.04 119.38))
     (stroke (width 0) (type default) (color 0 0 0 0))
@@
     (stroke (width 0) (type default) (color 0 0 0 0))
   )
-  (wire (pts (xy 193.04 114.3) (xy 193.04 119.38))
+  (wire (pts (xy 193.04 115.57) (xy 193.04 119.38))
     (stroke (width 0) (type default) (color 0 0 0 0))
   )
@@
   )
   (wire (pts (xy 129.54 134.62) (xy 140.97 134.62))
+    (stroke (width 0) (type default) (color 0 0 0 0))
+  )
+  (wire (pts (xy 77.47 91.44) (xy 77.47 105.41))
     (stroke (width 0) (type default) (color 0 0 0 0))
   )
@@
     (effects (font (size 1.27 1.27)) (justify left bottom))
   )
-  (global_label "12V" (shape input) (at 142.24 57.15 90) (fields_autoplaced)
+  (text "Etapa de potencia" (at 186.69 190.5 0)
+    (effects (font (size 1.27 1.27)) (justify left bottom))
+  )
+  (label "12V" (at 121.92 119.38 180)
+    (effects (font (size 1.27 1.27)) (justify right bottom))
+  )
+  (label "12V" (at 102.87 86.36 0)
+    (effects (font (size 1.27 1.27)) (justify left bottom))
+  )
+  (label "12V" (at 110.49 63.5 0)
+    (effects (font (size 1.27 1.27)) (justify left bottom))
+  )
+  (label "5V" (at 226.06 63.5 180)
+    (effects (font (size 1.27 1.27)) (justify right bottom))
+  )
+  (hierarchical_label "12V" (shape output) (at 99.06 81.28 90)
     (effects (font (size 1.27 1.27)) (justify left))
-    (property "Intersheet References" "${INTERSHEET_REFS}" (id 0) (at 142.1606 51.2293 90)
-      (effects (font (size 1.27 1.27)) (justify left) hide)
-    )
-  )
-  (global_label "5V" (shape input) (at 129.54 113.03 90) (fields_autoplaced)
+  )
+  (hierarchical_label "3.3V" (shape output) (at 193.04 115.57 90)
     (effects (font (size 1.27 1.27)) (justify left))
-    (property "Intersheet References" "${INTERSHEET_REFS}" (id 0) (at 129.4606 108.3188 90)
-      (effects (font (size 1.27 1.27)) (justify left) hide)
-    )
-  )
-  (global_label "5V" (shape input) (at 217.17 60.96 90) (fields_autoplaced)
+  )
+  (hierarchical_label "5V" (shape output) (at 217.17 60.96 90)
     (effects (font (size 1.27 1.27)) (justify left))
-    (property "Intersheet References" "${INTERSHEET_REFS}" (id 0) (at 217.0906 56.2488 90)
-      (effects (font (size 1.27 1.27)) (justify left) hide)
-    )
-  )
-  (global_label "3.3V" (shape input) (at 193.04 114.3 90) (fields_autoplaced)
-    (effects (font (size 1.27 1.27)) (justify left))
-    (property "Intersheet References" "${INTERSHEET_REFS}" (id 0) (at 192.9606 107.7745 90)
-      (effects (font (size 1.27 1.27)) (justify left) hide)
-    )
   )
   (symbol (lib_id "Device:C") (at 140.97 125.73 0) (unit 1)
@@
     (pin "3")
   )
+  (symbol (lib_id "Connector:Barrel_Jack") (at 64.77 88.9 0) (unit 1)
+    (in_bom yes) (on_board yes) (fields_autoplaced)
+    (property "Reference" "J?" (id 0) (at 64.77 80.01 0))
+    (property "Value" "Barrel_Jack" (id 1) (at 64.77 82.55 0))
+    (property "Footprint" "" (id 2) (at 66.04 89.916 0)
+      (effects (font (size 1.27 1.27)) hide)
+    )
+    (property "Datasheet" "~" (id 3) (at 66.04 89.916 0)
+      (effects (font (size 1.27 1.27)) hide)
+    )
+    (pin "1")
+    (pin "2")
+  )
   (symbol (lib_id "power:GND") (at 160.02 135.89 0) (unit 1)
     (in_bom yes) (on_board yes) (fields_autoplaced)
@@
     (pin "2")
   )
-  (symbol (lib_id "Switch:SW_DIP_x01") (at 102.87 63.5 0) (unit 1)
-    (in_bom yes) (on_board yes) (fields_autoplaced)
-    (property "Reference" "SW?" (id 0) (at 102.87 55.88 0))
-    (property "Value" "SW_DIP_x01" (id 1) (at 102.87 58.42 0))
-    (property "Footprint" "" (id 2) (at 102.87 63.5 0)
-      (effects (font (size 1.27 1.27)) hide)
-    )
-    (property "Datasheet" "~" (id 3) (at 102.87 63.5 0)
-      (effects (font (size 1.27 1.27)) hide)
-    )
-    (pin "1")
-    (pin "2")
-  )
   (symbol (lib_id "power:GND") (at 127 82.55 0) (unit 1)
     (in_bom yes) (on_board yes) (fields_autoplaced)
@@
     (pin "1")
     (pin "2")
-  )
-  (symbol (lib_id "power:Earth") (at 92.71 82.55 0) (unit 1)
-    (in_bom yes) (on_board yes) (fields_autoplaced)
-    (property "Reference" "#PWR?" (id 0) (at 92.71 88.9 0)
-      (effects (font (size 1.27 1.27)) hide)
-    )
-    (property "Value" "Earth" (id 1) (at 92.71 86.36 0)
-      (effects (font (size 1.27 1.27)) hide)
-    )
-    (property "Footprint" "" (id 2) (at 92.71 82.55 0)
-      (effects (font (size 1.27 1.27)) hide)
-    )
-    (property "Datasheet" "~" (id 3) (at 92.71 82.55 0)
-      (effects (font (size 1.27 1.27)) hide)
-    )
-    (pin "1")
   )
   (symbol (lib_id "Device:C_Polarized_US") (at 129.54 125.73 0) (unit 1)
@@
     (pin "1")
     (pin "2")
+  )
+  (symbol (lib_id "power:Earth") (at 77.47 105.41 0) (unit 1)
+    (in_bom yes) (on_board yes) (fields_autoplaced)
+    (property "Reference" "#PWR?" (id 0) (at 77.47 111.76 0)
+      (effects (font (size 1.27 1.27)) hide)
+    )
+    (property "Value" "Earth" (id 1) (at 77.47 109.22 0)
+      (effects (font (size 1.27 1.27)) hide)
+    )
+    (property "Footprint" "" (id 2) (at 77.47 105.41 0)
+      (effects (font (size 1.27 1.27)) hide)
+    )
+    (property "Datasheet" "~" (id 3) (at 77.47 105.41 0)
+      (effects (font (size 1.27 1.27)) hide)
+    )
+    (pin "1")
   )
   (symbol (lib_id "Device:C_Polarized_US") (at 193.04 125.73 0) (unit 1)
@@
     (pin "2")
   )
-  (symbol (lib_id "Connector:Barrel_Jack") (at 80.01 66.04 0) (unit 1)
-    (in_bom yes) (on_board yes) (fields_autoplaced)
-    (property "Reference" "J?" (id 0) (at 80.01 57.15 0))
-    (property "Value" "Barrel_Jack" (id 1) (at 80.01 59.69 0))
-    (property "Footprint" "" (id 2) (at 81.28 67.056 0)
-      (effects (font (size 1.27 1.27)) hide)
-    )
-    (property "Datasheet" "~" (id 3) (at 81.28 67.056 0)
-      (effects (font (size 1.27 1.27)) hide)
-    )
-    (pin "1")
-    (pin "2")
-  )
   (symbol (lib_id "power:GND") (at 217.17 83.82 0) (unit 1)
     (in_bom yes) (on_board yes) (fields_autoplaced)
@@
     (pin "1")
   )
+  (symbol (lib_id "Switch:SW_DIP_x01") (at 87.63 86.36 0) (unit 1)
+    (in_bom yes) (on_board yes) (fields_autoplaced)
+    (property "Reference" "SW?" (id 0) (at 87.63 78.74 0))
+    (property "Value" "SW_DIP_x01" (id 1) (at 87.63 81.28 0))
+    (property "Footprint" "" (id 2) (at 87.63 86.36 0)
+      (effects (font (size 1.27 1.27)) hide)
+    )
+    (property "Datasheet" "~" (id 3) (at 87.63 86.36 0)
+      (effects (font (size 1.27 1.27)) hide)
+    )
+    (pin "1")
+    (pin "2")
+  )
   (symbol (lib_id "Device:C_Polarized_US") (at 217.17 72.39 0) (unit 1)

Commit message: Actualización Potencia
21/09/2022
Parts:
- removed C1: 100nF, symbol Device:C
- removed C2, C?: 1000uF, symbol Device:C_Polarized_US
- removed C? (x2): 100n, symbol Device:C
- removed C? (x2): 22u, symbol Device:C_Polarized_US
- removed D1: 1N4007, Diode_THT:D_DO-41_SOD81_P10.16mm_Horizontal, symbol Diode:1N4007
- removed D?: BZT52Bxx, Diode_SMD:D_SOD-123F, symbol Diode:BZT52Bxx
- removed J?: Barrel_Jack, symbol Connector:Barrel_Jack
- removed L1: 68u, symbol Device:L
- removed R?: 10k, symbol Device:R
- removed R?: R, symbol Device:R
- removed SW?: SW_DIP_x01, symbol Switch:SW_DIP_x01
- removed U1: LM2596S-5, Package_TO_SOT_SMD:TO-263-5_TabPin3, symbol Regulator_Switching:LM2596S-5
- removed U?: AMS1117-3.3, Package_TO_SOT_SMD:SOT-223-3_TabPin2, symbol Regulator_Linear:AMS1117-3.3
- added C10: 100nF, symbol Device:C
- added C11: 1000uF, symbol Device:C_Polarized_US
- added C12: 10uF, symbol Device:C_Polarized_US
- added C13: 22uF, symbol Device:C_Polarized_US
- added C14, C15: 22u, symbol Device:C_Polarized_US
- added D?: 1N4007, Diode_THT:D_DO-41_SOD81_P10.16mm_Horizontal, symbol Diode:1N4007
- added J?: Barrel_Jack, symbol Connector:Barrel_Jack
- added SW?: SW_DIP_x01, symbol Switch:SW_DIP_x01
- added U?: AMS1117-5.0, Package_TO_SOT_SMD:SOT-223-3_TabPin2, symbol Regulator_Linear:AMS1117-5.0
- added U?: AMS1117-3.3, Package_TO_SOT_SMD:SOT-223-3_TabPin2, symbol Regulator_Linear:AMS1117-3.3
Connections:
- net 12V: now also C10.1, C11.1, C12.1, C14.1, D?.1 (K), U?.3 (VI), U?.3 (VI)
- net 3.3V: now also C15.1, U?.2 (VO)
- net 5V: now also C13.1, U?.2 (VO)
- net Earth: now also J?.2
- net GND: now also C10.2, C11.2, C12.2, C13.2, C14.2, C15.2, U?.1 (GND), U?.1 (GND)
- new net: J?.1, SW?.1
- new net: D?.2 (A), SW?.2
Other:
- note removed: "Diodo Zener SMD"
