File: Esquemáticos/ESP32/Programacion.kicad_sch (KiCad schematic)
At the start: 7 parts

Commit message: Cambios hechos al esquemático, faltan detalles
Revisar el discord para dejar todo al día con el feedback de hoy
Parts:
- added U?: ESP32-WROOM-32, RF_Module:ESP32-WROOM-32, symbol RF_Module:ESP32-WROOM-32
Connections:
- net 3.3V: now also U?.2 (VDD)
- net BOOT: now also U?.25 (IO0)
- net EN: now also U?.3 (EN)
- net GND: now also U?.1 (GND), U?.15 (GND), U?.38 (GND), U?.39 (GND)
- new net MISO: U?.31 (IO19)
- new net MOSI: U?.37 (IO23)
- new net RST: U?.36 (IO22)
- new net SCK: U?.30 (IO18)
- new net SS: U?.29 (IO5)
Other:
- note added: "Interfaz para depurar"
- moved on the sheet: C_BOOT, C_EN, R?, SW_BOOT, SW_EN

Commit message: actualizacion raul 3.0
Parts:
- added D1: Led_operacion, LED_SMD:LED_1206_3216Metric, symbol LED:IR26-21C_L110_TR8
- added D2: Led_holamundo, LED_SMD:LED_1206_3216Metric, symbol LED:IR26-21C_L110_TR8
Connections:
- net BOOT: now also D2.2 (A)
- net EN: now also D1.2 (A)
- net GND: now also D1.1 (K), D2.1 (K)
Other:
- note added: "Habría que cambiar los valores de las resistencias para que funcionen los LEDs, ver archivo de multisim"
- moved on the sheet: C_BOOT, C_EN, R?, SW_BOOT, SW_EN

Commit message: Support
Parts:
- gave numbers to parts that had none: 4
- renumbered C_BOOT to C_BOOT1, C_EN to C_EN1, SW_BOOT to SW_BOOT1, SW_EN to SW_EN1
Other:
- note added: "Colocarle nombres a los pines de ESP 32 y no GPIO X, porque no son pines de uso general sino particular. Ej. Al pin de SDA llamarle a su etiqueta "SDA" y no GPIO32"
- note added: "Ponerle condensadores de bypass a la entrada del ESP32 para eliminar armónicos de las señales múltiples que se trabajen"
Changed lines of the file:
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@@
+    (effects (font (size 1.27 1.27)) (justify left bottom))
+  )
+  (text "Ponerle condensadores de bypass a la entrada del ESP32 para eliminar armónicos de las señales múltiples que se trabajen\n"
+    (at 29.21 44.45 0)
+    (effects (font (size 1.27 1.27)) (justify left bottom))
+  )
+  (text "Colocarle nombres a los pines de ESP 32 y no GPIO X, porque no son pines de uso general sino particular. Ej. Al pin de SDA llamarle a su etiqueta \"SDA\" y no GPIO32"
+    (at 29.21 46.99 0)
     (effects (font (size 1.27 1.27)) (justify left bottom))
   )
@@
   (symbol (lib_id "power:GND") (at 151.13 124.46 0) (unit 1)
     (in_bom yes) (on_board yes) (fields_autoplaced)
-    (property "Reference" "#PWR?" (id 0) (at 151.13 130.81 0)
+    (property "Reference" "#PWR013" (id 0) (at 151.13 130.81 0)
       (effects (font (size 1.27 1.27)) hide)
     )
@@
   (symbol (lib_id "power:GND") (at 166.37 134.62 0) (unit 1)
     (in_bom yes) (on_board yes) (fields_autoplaced)
-    (property "Reference" "#PWR?" (id 0) (at 166.37 140.97 0)
+    (property "Reference" "#PWR014" (id 0) (at 166.37 140.97 0)
       (effects (font (size 1.27 1.27)) hide)
     )
@@
   (symbol (lib_id "RF_Module:ESP32-WROOM-32") (at 95.25 92.71 0) (unit 1)
     (in_bom yes) (on_board yes) (fields_autoplaced)
-    (property "Reference" "U?" (id 0) (at 97.2694 54.61 0)
+    (property "Reference" "U7" (id 0) (at 97.2694 54.61 0)
       (effects (font (size 1.27 1.27)) (justify left))
     )
@@
   (symbol (lib_id "power:GND") (at 243.84 135.89 0) (unit 1)
     (in_bom yes) (on_board yes) (fields_autoplaced)
-    (property "Reference" "#PWR?" (id 0) (at 243.84 142.24 0)
+    (property "Reference" "#PWR016" (id 0) (at 243.84 142.24 0)
       (effects (font (size 1.27 1.27)) hide)
     )
@@
   (symbol (lib_id "Device:R") (at 237.49 123.19 90) (unit 1)
     (in_bom yes) (on_board yes) (fields_autoplaced)
-    (property "Reference" "R?" (id 0) (at 237.49 116.84 90))
+    (property "Reference" "R26" (id 0) (at 237.49 116.84 90))
     (property "Value" "470" (id 1) (at 237.49 119.38 90))
     (property "Footprint" "" (id 2) (at 237.49 124.968 90)
@@
   (symbol (lib_id "Switch:SW_Push") (at 226.06 123.19 0) (unit 1)
     (in_bom yes) (on_board yes) (fields_autoplaced)
-    (property "Reference" "SW_BOOT" (id 0) (at 226.06 115.57 0))
+    (property "Reference" "SW_BOOT1" (id 0) (at 226.06 115.57 0))
     (property "Value" "SW_Push" (id 1) (at 226.06 118.11 0))
     (property "Footprint" "" (id 2) (at 226.06 118.11 0)
@@
   (symbol (lib_id "Switch:SW_Push") (at 158.75 121.92 0) (unit 1)
     (in_bom yes) (on_board yes) (fields_autoplaced)
-    (property "Reference" "SW_EN" (id 0) (at 158.75 114.3 0))
+    (property "Reference" "SW_EN1" (id 0) (at 158.75 114.3 0))
     (property "Value" "SW_Push" (id 1) (at 158.75 116.84 0))
     (property "Footprint" "" (id 2) (at 158.75 116.84 0)
@@
   (symbol (lib_id "Device:R") (at 250.19 109.22 90) (unit 1)
     (in_bom yes) (on_board yes) (fields_autoplaced)
-    (property "Reference" "R?" (id 0) (at 250.19 102.87 90))
+    (property "Reference" "R27" (id 0) (at 250.19 102.87 90))
     (property "Value" "10k" (id 1) (at 250.19 105.41 90))
     (property "Footprint" "" (id 2) (at 250.19 110.998 90)
@@
   (symbol (lib_id "power:GND") (at 218.44 125.73 0) (unit 1)
     (in_bom yes) (on_board yes) (fields_autoplaced)
-    (property "Reference" "#PWR?" (id 0) (at 218.44 132.08 0)
+    (property "Reference" "#PWR015" (id 0) (at 218.44 132.08 0)
       (effects (font (size 1.27 1.27)) hide)
     )
@@
   (symbol (lib_id "Device:R") (at 175.26 107.95 90) (unit 1)
     (in_bom yes) (on_board yes) (fields_autoplaced)
-    (property "Reference" "R?" (id 0) (at 175.26 101.6 90))
+    (property "Reference" "R25" (id 0) (at 175.26 101.6 90))
     (property "Value" "10k" (id 1) (at 175.26 104.14 90))
     (property "Footprint" "" (id 2) (at 175.26 109.728 90)
@@
   (symbol (lib_id "Device:C") (at 226.06 109.22 90) (unit 1)
     (in_bom yes) (on_board yes) (fields_autoplaced)
-    (property "Reference" "C_BOOT" (id 0) (at 226.06 101.6 90))
+    (property "Reference" "C_BOOT1" (id 0) (at 226.06 101.6 90))
     (property "Value" "100nF" (id 1) (at 226.06 104.14 90))
     (property "Footprint" "" (id 2) (at 229.87 108.2548 0)
@@
   (symbol (lib_id "Device:C") (at 158.75 107.95 90) (unit 1)
     (in_bom yes) (on_board yes) (fields_autoplaced)
-    (property "Reference" "C_EN" (id 0) (at 158.75 100.33 90))
+    (property "Reference" "C_EN1" (id 0) (at 158.75 100.33 90))
     (property "Value" "100nF" (id 1) (at 158.75 102.87 90))
     (property "Footprint" "" (id 2) (at 162.56 106.9848 0)

Commit message: auxilio
Parts:
- renumbered C_BOOT1 to C_BOOT, C_EN1 to C_EN, R26 to R?, R27 to R?, R25 to R?, SW_BOOT1 to SW_BOOT, SW_EN1 to SW_EN, U7 to U?
Other:
- note removed: "Colocarle nombres a los pines de ESP 32 y no GPIO X, porque no son pines de uso general sino particular. Ej. Al pin de SDA llamarle a su etiqueta "SDA" y no GPIO32"
- note removed: "Ponerle condensadores de bypass a la entrada del ESP32 para eliminar armónicos de las señales múltiples que se trabajen"
Changed lines of the file:
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@@
-    (effects (font (size 1.27 1.27)) (justify left bottom))
-  )
-  (text "Ponerle condensadores de bypass a la entrada del ESP32 para eliminar armónicos de las señales múltiples que se trabajen\n"
-    (at 29.21 44.45 0)
-    (effects (font (size 1.27 1.27)) (justify left bottom))
-  )
-  (text "Colocarle nombres a los pines de ESP 32 y no GPIO X, porque no son pines de uso general sino particular. Ej. Al pin de SDA llamarle a su etiqueta \"SDA\" y no GPIO32"
-    (at 29.21 46.99 0)
     (effects (font (size 1.27 1.27)) (justify left bottom))
   )
@@
   (symbol (lib_id "power:GND") (at 151.13 124.46 0) (unit 1)
     (in_bom yes) (on_board yes) (fields_autoplaced)
-    (property "Reference" "#PWR013" (id 0) (at 151.13 130.81 0)
+    (property "Reference" "#PWR?" (id 0) (at 151.13 130.81 0)
       (effects (font (size 1.27 1.27)) hide)
     )
@@
   (symbol (lib_id "power:GND") (at 166.37 134.62 0) (unit 1)
     (in_bom yes) (on_board yes) (fields_autoplaced)
-    (property "Reference" "#PWR014" (id 0) (at 166.37 140.97 0)
+    (property "Reference" "#PWR?" (id 0) (at 166.37 140.97 0)
       (effects (font (size 1.27 1.27)) hide)
     )
@@
   (symbol (lib_id "RF_Module:ESP32-WROOM-32") (at 95.25 92.71 0) (unit 1)
     (in_bom yes) (on_board yes) (fields_autoplaced)
-    (property "Reference" "U7" (id 0) (at 97.2694 54.61 0)
+    (property "Reference" "U?" (id 0) (at 97.2694 54.61 0)
       (effects (font (size 1.27 1.27)) (justify left))
     )
@@
   (symbol (lib_id "power:GND") (at 243.84 135.89 0) (unit 1)
     (in_bom yes) (on_board yes) (fields_autoplaced)
-    (property "Reference" "#PWR016" (id 0) (at 243.84 142.24 0)
+    (property "Reference" "#PWR?" (id 0) (at 243.84 142.24 0)
       (effects (font (size 1.27 1.27)) hide)
     )
@@
   (symbol (lib_id "Device:R") (at 237.49 123.19 90) (unit 1)
     (in_bom yes) (on_board yes) (fields_autoplaced)
-    (property "Reference" "R26" (id 0) (at 237.49 116.84 90))
+    (property "Reference" "R?" (id 0) (at 237.49 116.84 90))
     (property "Value" "470" (id 1) (at 237.49 119.38 90))
     (property "Footprint" "" (id 2) (at 237.49 124.968 90)
@@
   (symbol (lib_id "Switch:SW_Push") (at 226.06 123.19 0) (unit 1)
     (in_bom yes) (on_board yes) (fields_autoplaced)
-    (property "Reference" "SW_BOOT1" (id 0) (at 226.06 115.57 0))
+    (property "Reference" "SW_BOOT" (id 0) (at 226.06 115.57 0))
     (property "Value" "SW_Push" (id 1) (at 226.06 118.11 0))
     (property "Footprint" "" (id 2) (at 226.06 118.11 0)
@@
   (symbol (lib_id "Switch:SW_Push") (at 158.75 121.92 0) (unit 1)
     (in_bom yes) (on_board yes) (fields_autoplaced)
-    (property "Reference" "SW_EN1" (id 0) (at 158.75 114.3 0))
+    (property "Reference" "SW_EN" (id 0) (at 158.75 114.3 0))
     (property "Value" "SW_Push" (id 1) (at 158.75 116.84 0))
     (property "Footprint" "" (id 2) (at 158.75 116.84 0)
@@
   (symbol (lib_id "Device:R") (at 250.19 109.22 90) (unit 1)
     (in_bom yes) (on_board yes) (fields_autoplaced)
-    (property "Reference" "R27" (id 0) (at 250.19 102.87 90))
+    (property "Reference" "R?" (id 0) (at 250.19 102.87 90))
     (property "Value" "10k" (id 1) (at 250.19 105.41 90))
     (property "Footprint" "" (id 2) (at 250.19 110.998 90)
@@
   (symbol (lib_id "power:GND") (at 218.44 125.73 0) (unit 1)
     (in_bom yes) (on_board yes) (fields_autoplaced)
-    (property "Reference" "#PWR015" (id 0) (at 218.44 132.08 0)
+    (property "Reference" "#PWR?" (id 0) (at 218.44 132.08 0)
       (effects (font (size 1.27 1.27)) hide)
     )
@@
   (symbol (lib_id "Device:R") (at 175.26 107.95 90) (unit 1)
     (in_bom yes) (on_board yes) (fields_autoplaced)
-    (property "Reference" "R25" (id 0) (at 175.26 101.6 90))
+    (property "Reference" "R?" (id 0) (at 175.26 101.6 90))
     (property "Value" "10k" (id 1) (at 175.26 104.14 90))
     (property "Footprint" "" (id 2) (at 175.26 109.728 90)
@@
   (symbol (lib_id "Device:C") (at 226.06 109.22 90) (unit 1)
     (in_bom yes) (on_board yes) (fields_autoplaced)
-    (property "Reference" "C_BOOT1" (id 0) (at 226.06 101.6 90))
+    (property "Reference" "C_BOOT" (id 0) (at 226.06 101.6 90))
     (property "Value" "100nF" (id 1) (at 226.06 104.14 90))
     (property "Footprint" "" (id 2) (at 229.87 108.2548 0)
@@
   (symbol (lib_id "Device:C") (at 158.75 107.95 90) (unit 1)
     (in_bom yes) (on_board yes) (fields_autoplaced)
-    (property "Reference" "C_EN1" (id 0) (at 158.75 100.33 90))
+    (property "Reference" "C_EN" (id 0) (at 158.75 100.33 90))
     (property "Value" "100nF" (id 1) (at 158.75 102.87 90))
     (property "Footprint" "" (id 2) (at 162.56 106.9848 0)

Commit message: Mas commits :sunglasses:
Agragados números de los componentes
Parts:
- gave numbers to parts that had none: 4
- renumbered C_BOOT to C_BOOT1, C_EN to C_EN1, SW_BOOT to SW_BOOT1, SW_EN to SW_EN1
Changed lines of the file:
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@@
   (symbol (lib_id "power:GND") (at 151.13 124.46 0) (unit 1)
     (in_bom yes) (on_board yes) (fields_autoplaced)
-    (property "Reference" "#PWR?" (id 0) (at 151.13 130.81 0)
+    (property "Reference" "#PWR013" (id 0) (at 151.13 130.81 0)
       (effects (font (size 1.27 1.27)) hide)
     )
@@
   (symbol (lib_id "power:GND") (at 166.37 134.62 0) (unit 1)
     (in_bom yes) (on_board yes) (fields_autoplaced)
-    (property "Reference" "#PWR?" (id 0) (at 166.37 140.97 0)
+    (property "Reference" "#PWR014" (id 0) (at 166.37 140.97 0)
       (effects (font (size 1.27 1.27)) hide)
     )
@@
   (symbol (lib_id "RF_Module:ESP32-WROOM-32") (at 95.25 92.71 0) (unit 1)
     (in_bom yes) (on_board yes) (fields_autoplaced)
-    (property "Reference" "U?" (id 0) (at 97.2694 54.61 0)
+    (property "Reference" "U7" (id 0) (at 97.2694 54.61 0)
       (effects (font (size 1.27 1.27)) (justify left))
     )
@@
   (symbol (lib_id "power:GND") (at 243.84 135.89 0) (unit 1)
     (in_bom yes) (on_board yes) (fields_autoplaced)
-    (property "Reference" "#PWR?" (id 0) (at 243.84 142.24 0)
+    (property "Reference" "#PWR016" (id 0) (at 243.84 142.24 0)
       (effects (font (size 1.27 1.27)) hide)
     )
@@
   (symbol (lib_id "Device:R") (at 237.49 123.19 90) (unit 1)
     (in_bom yes) (on_board yes) (fields_autoplaced)
-    (property "Reference" "R?" (id 0) (at 237.49 116.84 90))
+    (property "Reference" "R26" (id 0) (at 237.49 116.84 90))
     (property "Value" "470" (id 1) (at 237.49 119.38 90))
     (property "Footprint" "" (id 2) (at 237.49 124.968 90)
@@
   (symbol (lib_id "Switch:SW_Push") (at 226.06 123.19 0) (unit 1)
     (in_bom yes) (on_board yes) (fields_autoplaced)
-    (property "Reference" "SW_BOOT" (id 0) (at 226.06 115.57 0))
+    (property "Reference" "SW_BOOT1" (id 0) (at 226.06 115.57 0))
     (property "Value" "SW_Push" (id 1) (at 226.06 118.11 0))
     (property "Footprint" "" (id 2) (at 226.06 118.11 0)
@@
   (symbol (lib_id "Switch:SW_Push") (at 158.75 121.92 0) (unit 1)
     (in_bom yes) (on_board yes) (fields_autoplaced)
-    (property "Reference" "SW_EN" (id 0) (at 158.75 114.3 0))
+    (property "Reference" "SW_EN1" (id 0) (at 158.75 114.3 0))
     (property "Value" "SW_Push" (id 1) (at 158.75 116.84 0))
     (property "Footprint" "" (id 2) (at 158.75 116.84 0)
@@
   (symbol (lib_id "Device:R") (at 250.19 109.22 90) (unit 1)
     (in_bom yes) (on_board yes) (fields_autoplaced)
-    (property "Reference" "R?" (id 0) (at 250.19 102.87 90))
+    (property "Reference" "R27" (id 0) (at 250.19 102.87 90))
     (property "Value" "10k" (id 1) (at 250.19 105.41 90))
     (property "Footprint" "" (id 2) (at 250.19 110.998 90)
@@
   (symbol (lib_id "power:GND") (at 218.44 125.73 0) (unit 1)
     (in_bom yes) (on_board yes) (fields_autoplaced)
-    (property "Reference" "#PWR?" (id 0) (at 218.44 132.08 0)
+    (property "Reference" "#PWR015" (id 0) (at 218.44 132.08 0)
       (effects (font (size 1.27 1.27)) hide)
     )
@@
   (symbol (lib_id "Device:R") (at 175.26 107.95 90) (unit 1)
     (in_bom yes) (on_board yes) (fields_autoplaced)
-    (property "Reference" "R?" (id 0) (at 175.26 101.6 90))
+    (property "Reference" "R25" (id 0) (at 175.26 101.6 90))
     (property "Value" "10k" (id 1) (at 175.26 104.14 90))
     (property "Footprint" "" (id 2) (at 175.26 109.728 90)
@@
   (symbol (lib_id "Device:C") (at 226.06 109.22 90) (unit 1)
     (in_bom yes) (on_board yes) (fields_autoplaced)
-    (property "Reference" "C_BOOT" (id 0) (at 226.06 101.6 90))
+    (property "Reference" "C_BOOT1" (id 0) (at 226.06 101.6 90))
     (property "Value" "100nF" (id 1) (at 226.06 104.14 90))
     (property "Footprint" "" (id 2) (at 229.87 108.2548 0)
@@
   (symbol (lib_id "Device:C") (at 158.75 107.95 90) (unit 1)
     (in_bom yes) (on_board yes) (fields_autoplaced)
-    (property "Reference" "C_EN" (id 0) (at 158.75 100.33 90))
+    (property "Reference" "C_EN1" (id 0) (at 158.75 100.33 90))
     (property "Value" "100nF" (id 1) (at 158.75 102.87 90))
     (property "Footprint" "" (id 2) (at 162.56 106.9848 0)

Commit message: Push mid :V
Other:
- note added: "Colocarle nombres a los pines de ESP 32 y no GPIO X, porque no son pines de uso general sino particular. Ej. Al pin de SDA llamarle a su etiqueta "SDA" y no GPIO32"
- note added: "Ponerle condensadores de bypass a la entrada del ESP32 para eliminar armónicos de las señales múltiples que se trabajen"
Changed lines of the file:
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@@
+    (effects (font (size 1.27 1.27)) (justify left bottom))
+  )
+  (text "Ponerle condensadores de bypass a la entrada del ESP32 para eliminar armónicos de las señales múltiples que se trabajen\n"
+    (at 29.21 44.45 0)
+    (effects (font (size 1.27 1.27)) (justify left bottom))
+  )
+  (text "Colocarle nombres a los pines de ESP 32 y no GPIO X, porque no son pines de uso general sino particular. Ej. Al pin de SDA llamarle a su etiqueta \"SDA\" y no GPIO32"
+    (at 29.21 46.99 0)
     (effects (font (size 1.27 1.27)) (justify left bottom))
   )
