File: Esquemáticos/ESP32/Programacion.kicad_sch (KiCad schematic)
At the start: 13 parts, among them J4 USB Programador, U7 ESP32-WROOM-32

Commit message: Actualizadas las huellas de R y C
De acuerdo con la recomendación del profe, ahora todas son 0603.
Parts:
- C_BOOT1, C_RST1: footprint Capacitor_SMD:C_0201_0603Metric_Pad0.64x0.40mm_HandSolder -> Capacitor_SMD:C_0603_1608Metric_Pad1.08x0.95mm_HandSolder
- D2: footprint LED_SMD:LED_1206_3216Metric -> LED_SMD:LED_0603_1608Metric_Pad1.05x0.95mm_HandSolder
- R25, R26, R27, R28, RRX1, RTX1: footprint Resistor_SMD:R_1206_3216Metric_Pad1.30x1.75mm_HandSolder -> Resistor_SMD:R_0603_1608Metric_Pad0.98x0.95mm_HandSolder
Changed lines of the file:
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@@
     (property "Reference" "RRX1" (id 0) (at 143.51 74.93 90))
     (property "Value" "R" (id 1) (at 143.51 77.47 90))
-    (property "Footprint" "Resistor_SMD:R_1206_3216Metric_Pad1.30x1.75mm_HandSolder" (id 2) (at 143.51 74.168 90)
+    (property "Footprint" "Resistor_SMD:R_0603_1608Metric_Pad0.98x0.95mm_HandSolder" (id 2) (at 143.51 74.168 90)
       (effects (font (size 1.27 1.27)) hide)
     )
@@
     (property "Reference" "R26" (id 0) (at 237.49 116.84 90))
     (property "Value" "470" (id 1) (at 237.49 119.38 90))
-    (property "Footprint" "Resistor_SMD:R_1206_3216Metric_Pad1.30x1.75mm_HandSolder" (id 2) (at 237.49 124.968 90)
+    (property "Footprint" "Resistor_SMD:R_0603_1608Metric_Pad0.98x0.95mm_HandSolder" (id 2) (at 237.49 124.968 90)
       (effects (font (size 1.27 1.27)) hide)
     )
@@
     (property "Reference" "RTX1" (id 0) (at 143.51 64.77 90))
     (property "Value" "R" (id 1) (at 143.51 67.31 90))
-    (property "Footprint" "Resistor_SMD:R_1206_3216Metric_Pad1.30x1.75mm_HandSolder" (id 2) (at 143.51 71.628 90)
+    (property "Footprint" "Resistor_SMD:R_0603_1608Metric_Pad0.98x0.95mm_HandSolder" (id 2) (at 143.51 71.628 90)
       (effects (font (size 1.27 1.27)) hide)
     )
@@
     (property "Reference" "R27" (id 0) (at 250.19 102.87 90))
     (property "Value" "10k" (id 1) (at 250.19 105.41 90))
-    (property "Footprint" "Resistor_SMD:R_1206_3216Metric_Pad1.30x1.75mm_HandSolder" (id 2) (at 250.19 110.998 90)
+    (property "Footprint" "Resistor_SMD:R_0603_1608Metric_Pad0.98x0.95mm_HandSolder" (id 2) (at 250.19 110.998 90)
       (effects (font (size 1.27 1.27)) hide)
     )
@@
       (effects (font (size 1.27 1.27)) (justify right))
     )
-    (property "Footprint" "LED_SMD:LED_1206_3216Metric" (id 2) (at 115.57 119.38 0)
+    (property "Footprint" "LED_SMD:LED_0603_1608Metric_Pad1.05x0.95mm_HandSolder" (id 2) (at 115.57 119.38 0)
       (effects (font (size 1.27 1.27)) hide)
     )
@@
     (property "Reference" "R25" (id 0) (at 175.26 101.6 90))
     (property "Value" "10k" (id 1) (at 175.26 104.14 90))
-    (property "Footprint" "Resistor_SMD:R_1206_3216Metric_Pad1.30x1.75mm_HandSolder" (id 2) (at 175.26 109.728 90)
+    (property "Footprint" "Resistor_SMD:R_0603_1608Metric_Pad0.98x0.95mm_HandSolder" (id 2) (at 175.26 109.728 90)
       (effects (font (size 1.27 1.27)) hide)
     )
@@
     (property "Reference" "R28" (id 0) (at 116.84 106.68 90))
     (property "Value" "56" (id 1) (at 116.84 109.22 90))
-    (property "Footprint" "Resistor_SMD:R_1206_3216Metric_Pad1.30x1.75mm_HandSolder" (id 2) (at 116.84 114.808 90)
+    (property "Footprint" "Resistor_SMD:R_0603_1608Metric_Pad0.98x0.95mm_HandSolder" (id 2) (at 116.84 114.808 90)
       (effects (font (size 1.27 1.27)) hide)
     )
@@
     (property "Reference" "C_BOOT1" (id 0) (at 226.06 101.6 90))
     (property "Value" "100nF" (id 1) (at 226.06 104.14 90))
-    (property "Footprint" "Capacitor_SMD:C_0201_0603Metric_Pad0.64x0.40mm_HandSolder" (id 2) (at 229.87 108.2548 0)
+    (property "Footprint" "Capacitor_SMD:C_0603_1608Metric_Pad1.08x0.95mm_HandSolder" (id 2) (at 229.87 108.2548 0)
       (effects (font (size 1.27 1.27)) hide)
     )
@@
     (property "Reference" "C_RST1" (id 0) (at 158.75 100.33 90))
     (property "Value" "100nF" (id 1) (at 158.75 102.87 90))
-    (property "Footprint" "Capacitor_SMD:C_0201_0603Metric_Pad0.64x0.40mm_HandSolder" (id 2) (at 162.56 106.9848 0)
-      (effects (font (size 1.27 1.27)) hide)
-    )
+    (property "Footprint" "Capacitor_SMD:C_0603_1608Metric_Pad1.08x0.95mm_HandSolder" (id 2) (at 162.56 106.9848 0)
+      (effects (font (size 1.27 1.27)) hide)
+    )
