File: Esquemáticos/ESP32/RFID.kicad_sch (KiCad schematic)
At the start: 1 part, among them U8 RFID_RC522

Commit message: auxilio
Parts:
- renumbered U8 to U1
Changed lines of the file:
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@@
   (symbol (lib_id "libreria_raul:RFID_RC522") (at 149.86 93.98 0) (unit 1)
     (in_bom yes) (on_board yes) (fields_autoplaced)
-    (property "Reference" "U8" (id 0) (at 163.83 101.5999 0)
+    (property "Reference" "U1" (id 0) (at 163.83 101.5999 0)
       (effects (font (size 1.27 1.27)) (justify left))
     )
@@
   (symbol (lib_id "power:GND") (at 134.62 104.14 270) (unit 1)
     (in_bom yes) (on_board yes) (fields_autoplaced)
-    (property "Reference" "#PWR012" (id 0) (at 128.27 104.14 0)
+    (property "Reference" "#PWR?" (id 0) (at 128.27 104.14 0)
       (effects (font (size 1.27 1.27)) hide)
     )
